File: hardware/bottom-r1.sch (EAGLE design)
At the start: 47 parts, among them J1 BOTTOM, J2 RTD, J3 TC1, J4 TC2, J5 TC3, U1 ADS1248, U2 MS5803-14BA, U3 HIH6131

Commit message: Route bottom sensors PCB, please review
Parts:
- removed R10, R12, R2, R9: 10K, SparkFun-Passives:RESISTOR0805-RES
- added L2: FERRITE, HAB:INDUCTOR1206
- C3: value 10u -> 1u
Connections:
- removed net CLK: R2.2, U1.CLK
- net 3.3V: now also L2.2; no longer R10.2, R12.2, R9.2
- net AVDD: now also L2.1
- net CSADC: no longer R9.1
- net CSHUM: no longer R12.1
- net CSPRS: no longer R10.1
- net GND: now also U1.CLK; no longer R2.1
- net RTD1: now also J2.2; no longer J2.1
- net RTD2: now also J2.1; no longer J2.2
- net TC1N: now also J3.3; no longer J3.1
- net TC1P: now also J3.1; no longer J3.3
- net TC2N: now also J4.3; no longer J4.1
- net TC2P: now also J4.1; no longer J4.3
- net TC3N: now also J5.3; no longer J5.1
- net TC3P: now also J5.1; no longer J5.3
