File: hardware/telemetry-b1.sch (EAGLE design)
At the start: 115 parts, among them IC1 COPERNICUSSMD, IC10 TPS70933, IC2 TPS70933, IC4 STM32L073CZT6, IC5 TPS62160, IC6 HX1, IC7 LMP7702, J1 I2C, J10 TEMP_BAT, J11 DNP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

Commit message: Fix I2C pull-up resistors in beta/regular boards; add Phoenix board and some datasheets
Parts:
- added R10, R21: 4.7K, SparkFun-Passives:RESISTOR0805-RES
Connections:
- net 3.3V: now also R10.1, R21.1
- net SCL: now also R21.2
- net SDA: now also R10.2
Other:
- note added: "2"
- note removed: "1"
Changed lines of the file:
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@@
 <part name="R34" library="SparkFun-Passives" deviceset="RESISTOR" device="0805-RES" value="1"/>
 <part name="JP4" library="SparkFun-Connectors" deviceset="M02" device="PTH" value="BAT2"/>
+<part name="R21" library="SparkFun-Passives" deviceset="RESISTOR" device="0805-RES" value="4.7K"/>
+<part name="R10" library="SparkFun-Passives" deviceset="RESISTOR" device="0805-RES" value="4.7K"/>
+<part name="SUPPLY23" library="SparkFun-Aesthetics" deviceset="3.3V" device=""/>
 </parts>
 <sheets>
@@
 <plain>
 <text x="152.4" y="7.62" size="2.54" layer="94">Stephen Carlson</text>
-<text x="236.22" y="7.62" size="2.54" layer="94">1</text>
+<text x="236.22" y="7.62" size="2.54" layer="94">2</text>
 <text x="38.1" y="129.54" size="1.778" layer="90">535-10241-1-ND</text>
 <text x="7.62" y="129.54" size="1.778" layer="90">887-1233-ND</text>
@@
 <wire x1="332.74" y1="53.34" x2="403.86" y2="53.34" width="0.3048" layer="94"/>
 <wire x1="403.86" y1="53.34" x2="403.86" y2="106.68" width="0.3048" layer="94"/>
-<text x="497.84" y="7.62" size="2.54" layer="94">1</text>
+<text x="497.84" y="7.62" size="2.54" layer="94">2</text>
 <wire x1="403.86" y1="53.34" x2="408.94" y2="53.34" width="0.3048" layer="94"/>
 <wire x1="408.94" y1="53.34" x2="408.94" y2="35.56" width="0.3048" layer="94"/>
@@
 <instance part="JP4" gate="G$1" x="327.66" y="88.9" rot="MR0"/>
 <instance part="R2" gate="A" x="111.76" y="170.18" rot="R270"/>
+<instance part="R21" gate="G$1" x="228.6" y="170.18" rot="R270"/>
+<instance part="R10" gate="G$1" x="238.76" y="170.18" rot="R270"/>
+<instance part="SUPPLY23" gate="G$1" x="233.68" y="177.8"/>
 </instances>
 <busses>
@@
 <junction x="299.72" y="78.74"/>
 </segment>
+<segment>
+<pinref part="R21" gate="G$1" pin="1"/>
+<pinref part="R10" gate="G$1" pin="1"/>
+<wire x1="228.6" y1="175.26" x2="233.68" y2="175.26" width="0.1524" layer="91"/>
+<pinref part="SUPPLY23" gate="G$1" pin="3.3V"/>
+<wire x1="233.68" y1="175.26" x2="238.76" y2="175.26" width="0.1524" layer="91"/>
+<wire x1="233.68" y1="177.8" x2="233.68" y2="175.26" width="0.1524" layer="91"/>
+<junction x="233.68" y="175.26"/>
+</segment>
 </net>
 <net name="VDDA" class="0">
@@
 <label x="269.24" y="81.28" size="1.778" layer="95"/>
 </segment>
+<segment>
+<pinref part="R21" gate="G$1" pin="2"/>
+<wire x1="223.52" y1="162.56" x2="228.6" y2="162.56" width="0.1524" layer="91"/>
+<wire x1="228.6" y1="162.56" x2="228.6" y2="165.1" width="0.1524" layer="91"/>
+<label x="223.52" y="162.56" size="1.778" layer="95"/>
+</segment>
 </net>
 <net name="SDA" class="0">
@@
 <label x="269.24" y="86.36" size="1.778" layer="95"/>
 </segment>
-</net>
+<segment>
+<pinref part="R10" gate="G$1" pin="2"/>
+<wire x1="223.52" y1="160.02" x2="238.76" y2="160.02" width="0.1524" layer="91"/>
+<wire x1="238.76" y1="160.02" x2="238.76" y2="165.1" width="0.1524" layer="91"/>
+<label x="223.52" y="160.02" size="1.778" layer="95"/>
+</segment>
+</net>
