File: hardware/lora-rx.sch (EAGLE design)
At the start: 31 parts, among them J1 USB-A-H, J2 SMA_EDGE, J3 DNP, U1 STM32L052K8, U2 SX1278, U3 TPS70933

Commit message: Commit a few outstanding clean-up changes (not integrated into actual hardware) left in the current directory
Other:
- note removed: "TODO Adjust resistors based on OTRTAll"
Changed lines of the file:
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@@
 <plain>
 <text x="55.88" y="101.6" size="1.778" layer="90">497-14904-ND</text>
-<text x="124.46" y="99.06" size="1.778" layer="90">TODO Adjust resistors based on OTRTAll</text>
 <text x="149.86" y="7.62" size="2.54" layer="94">Phoenix</text>
 <text x="236.22" y="7.62" size="2.54" layer="94">A</text>
