File: hardware/telemetry-phoenix.brd (EAGLE design)
At the start: 65 x 56 mm, 113 parts, among them IC10 TPS70933, IC11 VN5160S-E, IC2 TPS70933, IC3 BME280, IC4 STM32L052C8T6, IC5 TPS62160, IC6 HX1, IC7 LMP7702, IC8 ADXL345, IC9 VN5160S-E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

Commit message: Commit a few outstanding clean-up changes (not integrated into actual hardware) left in the current directory
Parts:
- moved R7 7.10 mm to (41.3, 36.8), turned to 180 degrees
Connections:
- net 3.3V: no longer R26.2
- net GND: now also R26.2
Routing:
- net BTN: track 19.4 -> 28.3 mm
- net 3.3V: track 45.0 -> 40.1 mm
Changed lines of the file:
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@@
 <attribute name="VALUE" x="39.751" y="31.242" size="0.6096" layer="27" ratio="15" rot="R180"/>
 </element>
-<element name="R7" library="SparkFun-Passives" package="0805" value="10K" x="44.45" y="43.18" smashed="yes" rot="R270">
-<attribute name="NAME" x="44.577" y="41.7195" size="0.6096" layer="25" ratio="15" rot="R180"/>
-<attribute name="VALUE" x="43.053" y="44.196" size="0.6096" layer="27" ratio="15" rot="R270"/>
+<element name="R7" library="SparkFun-Passives" package="0805" value="10K" x="41.275" y="36.83" smashed="yes" rot="R180">
+<attribute name="NAME" x="39.8145" y="36.703" size="0.6096" layer="25" ratio="15" rot="R90"/>
+<attribute name="VALUE" x="42.291" y="38.227" size="0.6096" layer="27" ratio="15" rot="R180"/>
 </element>
 <element name="R8" library="SparkFun-Passives" package="0805" value="DNP" x="17.78" y="46.99" smashed="yes">
@@
 <contactref element="C13" pad="1"/>
 <contactref element="R6" pad="2"/>
-<contactref element="R26" pad="2"/>
 <contactref element="R7" pad="2"/>
 <contactref element="R5" pad="2"/>
@@
 <vertex x="34.925" y="30.48"/>
 <vertex x="34.925" y="36.83"/>
-<vertex x="39.37" y="36.83"/>
-<vertex x="39.37" y="34.29"/>
-<vertex x="40.005" y="34.29"/>
+<vertex x="40.005" y="36.83"/>
 <vertex x="40.005" y="37.465"/>
 <vertex x="36.83" y="37.465"/>
@@
 <wire x1="59.69" y1="35.56" x2="62.23" y2="35.56" width="0.4064" layer="1"/>
 <contactref element="J1" pad="4"/>
-<wire x1="44.45" y1="42.28" x2="44.45" y2="39.37" width="0.4064" layer="1"/>
-<wire x1="44.45" y1="39.37" x2="42.545" y2="37.465" width="0.4064" layer="1"/>
-<wire x1="42.545" y1="37.465" x2="41.275" y2="36.195" width="0.4064" layer="1"/>
-<wire x1="41.275" y1="36.195" x2="40.005" y2="36.195" width="0.4064" layer="1"/>
 <wire x1="23.865" y1="40.005" x2="23.865" y2="41.01" width="0.4064" layer="1"/>
 <wire x1="59.69" y1="35.56" x2="57.785" y2="33.655" width="0.4064" layer="1"/>
 <wire x1="57.785" y1="33.655" x2="55.88" y2="33.655" width="0.4064" layer="1"/>
 <via x="55.88" y="33.655" extent="1-16" drill="0.5"/>
-<wire x1="55.88" y1="33.655" x2="52.07" y2="37.465" width="0.4064" layer="16"/>
-<wire x1="52.07" y1="37.465" x2="42.545" y2="37.465" width="0.4064" layer="16"/>
-<via x="42.545" y="37.465" extent="1-16" drill="0.6"/>
+<via x="38.735" y="37.211" extent="1-16" drill="0.6"/>
 <wire x1="24.5" y1="43.815" x2="24.5" y2="41.645" width="0.4064" layer="1"/>
 <wire x1="24.5" y1="41.645" x2="23.865" y2="41.01" width="0.4064" layer="1"/>
@@
 <wire x1="24.5" y1="45.35" x2="22.86" y2="46.99" width="0.4064" layer="1"/>
 <wire x1="22.86" y1="46.99" x2="22.73" y2="46.99" width="0.4064" layer="1"/>
+<wire x1="38.735" y1="37.211" x2="52.324" y2="37.211" width="0.4064" layer="16"/>
+<wire x1="52.324" y1="37.211" x2="55.88" y2="33.655" width="0.4064" layer="16"/>
 </signal>
 <signal name="GND">
@@
 <wire x1="32.095" y1="29.155" x2="32.095" y2="27.595" width="0.2032" layer="1"/>
 <wire x1="32.095" y1="27.595" x2="32.385" y2="27.305" width="0.2032" layer="1"/>
-<via x="38.735" y="36.195" extent="1-16" drill="0.5"/>
-<via x="41.275" y="38.1" extent="1-16" drill="0.5"/>
+<via x="40.894" y="35.306" extent="1-16" drill="0.5"/>
+<via x="43.815" y="40.64" extent="1-16" drill="0.5"/>
 <contactref element="J5" pad="2"/>
 <wire x1="31.115" y1="22.987" x2="31.115" y2="22.86" width="0.4064" layer="1"/>
@@
 <vertex x="22.225" y="17.145"/>
 </polygon>
+<contactref element="R26" pad="2"/>
 </signal>
 <signal name="VDDA">
@@
 <contactref element="IC4" pad="41"/>
 <contactref element="R25" pad="2"/>
-<wire x1="34.345" y1="32.905" x2="39.255" y2="32.905" width="0.2032" layer="1"/>
-<wire x1="39.255" y1="32.905" x2="50.165" y2="43.815" width="0.2032" layer="1"/>
-<wire x1="50.165" y1="43.815" x2="53.075" y2="43.815" width="0.2032" layer="1"/>
+<wire x1="34.345" y1="32.905" x2="39.89" y2="32.905" width="0.2032" layer="1"/>
+<wire x1="39.89" y1="32.905" x2="50.8" y2="43.815" width="0.2032" layer="1"/>
+<wire x1="50.8" y1="43.815" x2="53.075" y2="43.815" width="0.2032" layer="1"/>
 </signal>
 <signal name="MISO">
 <contactref element="IC4" pad="40"/>
 <contactref element="R28" pad="2"/>
-<wire x1="34.345" y1="32.405" x2="40.66" y2="32.405" width="0.2032" layer="1"/>
-<wire x1="40.66" y1="32.405" x2="45.72" y2="37.465" width="0.2032" layer="1"/>
-<wire x1="45.72" y1="37.465" x2="48.26" y2="37.465" width="0.2032" layer="1"/>
+<wire x1="34.345" y1="32.405" x2="41.295" y2="32.405" width="0.2032" layer="1"/>
+<wire x1="41.295" y1="32.405" x2="46.355" y2="37.465" width="0.2032" layer="1"/>
+<wire x1="46.355" y1="37.465" x2="48.26" y2="37.465" width="0.2032" layer="1"/>
 <wire x1="48.26" y1="37.465" x2="50.8" y2="40.005" width="0.2032" layer="1"/>
 <wire x1="50.8" y1="40.005" x2="53.075" y2="40.005" width="0.2032" layer="1"/>
@@
 <contactref element="IC4" pad="39"/>
 <contactref element="R4" pad="2"/>
-<wire x1="34.345" y1="31.905" x2="42.065" y2="31.905" width="0.2032" layer="1"/>
-<wire x1="53.075" y1="36.195" x2="46.355" y2="36.195" width="0.2032" layer="1"/>
-<wire x1="46.355" y1="36.195" x2="42.065" y2="31.905" width="0.2032" layer="1"/>
+<wire x1="34.345" y1="31.905" x2="42.7" y2="31.905" width="0.2032" layer="1"/>
+<wire x1="53.075" y1="36.195" x2="46.99" y2="36.195" width="0.2032" layer="1"/>
+<wire x1="46.99" y1="36.195" x2="42.7" y2="31.905" width="0.2032" layer="1"/>
 </signal>
 <signal name="GPSTX">
@@
 <wire x1="34.29" y1="39.37" x2="38.0238" y2="39.37" width="0.2032" layer="16"/>
 <wire x1="38.0238" y1="39.37" x2="45.0088" y2="46.355" width="0.2032" layer="16"/>
-<wire x1="44.45" y1="44.08" x2="44.45" y2="45.7962" width="0.2032" layer="1"/>
 <wire x1="44.45" y1="45.7962" x2="45.0088" y2="46.355" width="0.2032" layer="1"/>
+<wire x1="45.0088" y1="46.355" x2="45.0088" y2="39.6638" width="0.2032" layer="1"/>
+<wire x1="42.175" y1="36.83" x2="45.0088" y2="39.6638" width="0.2032" layer="1"/>
 </signal>
 <signal name="B_MISO">

Commit message: Update schematic to hopefully fix phase angle issues with pre-emphasis filter
Parts:
- C25: value 330p -> 100p
- R56: value 430K -> 330K
Changed lines of the file:
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@@
 <attribute name="VALUE" x="44.958" y="18.161" size="0.6096" layer="27" ratio="15" rot="R270"/>
 </element>
-<element name="C25" library="SparkFun-Passives" package="0805" value="330p" x="19.685" y="36.195" smashed="yes" rot="R180">
+<element name="C25" library="SparkFun-Passives" package="0805" value="100p" x="19.685" y="36.195" smashed="yes" rot="R180">
 <attribute name="NAME" x="22.352" y="35.3695" size="0.6096" layer="25" ratio="15" rot="R180"/>
 <attribute name="VALUE" x="20.701" y="37.592" size="0.6096" layer="27" ratio="15" rot="R180"/>
@@
 <attribute name="VALUE" x="25.527" y="26.289" size="0.6096" layer="27" ratio="15" rot="R90"/>
 </element>
-<element name="R56" library="SparkFun-Passives" package="0805" value="430K" x="21.59" y="43.18" smashed="yes" rot="R270">
+<element name="R56" library="SparkFun-Passives" package="0805" value="330K" x="21.59" y="43.18" smashed="yes" rot="R270">
 <attribute name="NAME" x="20.828" y="44.6405" size="0.6096" layer="25" ratio="15"/>
 <attribute name="VALUE" x="22.733" y="44.196" size="0.6096" layer="27" ratio="15" rot="R270"/>
