File: hardware/telemetry-phoenix.sch (EAGLE design)
At the start: 110 parts, among them IC1 COPERNICUSSMD, IC10 TPS70933, IC2 TPS70933, IC3 74HC137, IC4 STM32L073CZT6, IC5 TPS62160, IC6 HX1, IC7 LMP7702, IC8 ADXL345, IC9 HIH9131, J1 I2C1, J10 TEMP_BAT, J11 DNP, J12 PHOTO_GP2, J13 LORA, J2 I2C2, J3 BOTTOM, J4 USD-SOCKET, J5 BAT, J6 SMA_EDGE, J7 SMA_EDGE, J8 TEMP_GPS, J9 PHOTO_GP4, Y1 32768, Y2 8M

Commit message: Fix I2C pull-up resistors in beta/regular boards; add Phoenix board and some datasheets
Parts:
- removed C31, C32, C33: 0.1u, SparkFun-Passives:CAP0805
- removed IC3: 74HC137, HAB:74LS137PW
- removed IC9: HIH9131, SparkFun-AnalogIC:HIH6131
- removed J10: TEMP_BAT, SparkFun-Connectors:M03JST-PTH
- removed J12: PHOTO_GP2, SparkFun-Connectors:M03JST-PTH
- removed J3: BOTTOM, SparkFun-Connectors:M102MM
- removed J4: USD-SOCKET, SparkFun-Connectors:USD-SOCKET
- removed J9: PHOTO_GP4, SparkFun-Connectors:M03JST-PTH
- added D12, D13: 15V, SparkFun-DiscreteSemi:DIODE-ZENER5.6V
- added FRAME3: FRAME-LETTERNO_PACKAGE, SparkFun-Aesthetics:FRAME-LETTERNO_PACKAGE
- added JP3: SDA, SparkFun-Passives:JUMPER-PAD-2-NC_BY_TRACE
- added JP4: SCL, SparkFun-Passives:JUMPER-PAD-2-NC_BY_TRACE
- added OK1, OK2, OK3: LTV826S, optocoupler:LTV826S
- added Q1: SI4202DY, HAB:SI4202DY
- added R30, R31, R32, R33, R34, R35, R36, R37, R38, R39: 4.7K, SparkFun-Passives:RESISTOR0805-RES
- added R40: 430K, SparkFun-Passives:RESISTOR0805-RES
- added R41, R46, R47: 100K, SparkFun-Passives:RESISTOR0805-RES
- added R42, R43, R44, R45, R48, R49, R50, R51: 10K, SparkFun-Passives:RESISTOR0805-RES
- added U1, U3: VN5160S-E, HAB:VN5160S-E
- added U2: BME280, BME280ComponentLibrary:BME280
- C27: value 0.1u -> 1u
- D1: value 12V -> 15V
- D6: value CM1213A -> 5.6V; device HAB:CM1213A -> SparkFun-DiscreteSemi:DIODE-ZENER5.6V
- IC4: value STM32L073CZT6 -> STM32L052C8T6
- J2: value I2C2 -> RASPBERRYPI-GPIOPTH; device SparkFun-Connectors:I2C_STANDARD_NO_SILK -> SparkFun-Boards:RASPBERRYPI-GPIOPTH
- J8: value TEMP_GPS -> TEMP_E
- R19: value 470K -> 430K
- R20: value 180K -> 100K
- R28: value 10K -> 0
- R3: value 100 -> 10K; device SparkFun-Passives:RESISTOR-ARRAY0603-ARV -> SparkFun-Passives:RESISTOR0805-RES
- R5, R8: value 100 -> DNP
Connections:
- net +9V renamed VBAT
- removed net AL_L: IC9.AL_L
- removed net B_CSADC: J3.7, R3B.1
- removed net B_CSHUM: J3.3, R3D.1
- removed net B_CSPRS: J3.6, R3C.1
- removed net CSA0: IC3A.A, IC4.PB7
- removed net CSA1: IC3A.B, IC4.PB6
- removed net CSA2: IC3A.C, IC4.PB12
- removed net CSADC: IC3A.Y5, R3B.2
- removed net CSBHUM: IC3A.Y3, R3D.2
- removed net CSHUM: IC3A.Y2, IC9.SCL
- removed net CSLAT: IC3A.GL, IC4.PA15, R6.1
- removed net CSLORA: IC3A.Y1, R22.1
- removed net CSPRS: IC3A.Y4, R3C.2
- removed net CSSD: IC3A.Y0, J4.CS
- removed net D+: IC4.PA12
- removed net D-: IC4.PA11
- removed net MCO: IC4.PA8
- removed net PHOTO_GP2: D6.CH2, IC4.PA5, J12.3
- removed net PHOTO_GP4: D6.CH1, IC4.PA2, J9.3
- removed net TEMPB: D6.CH4, IC4.PA1, J10.3
- removed net TEMPG: D6.CH3, IC4.PA0, J8.3
- removed net USIN: IC4.PB14
- removed net USOUT: IC4.PB15
- removed net USRES: IC4.PB13
- removed net VCORE: C28.1, IC9.VCORE
- new net 15V: C29.1, R40.2, U3.VCC
- new net 15V_OUT: U3.OUTPUT
- new net 5V_PI: C27.1, J2.5V@2, J2.5V@4, U1.OUTPUT
- new net ALT_CTRL: D13.C, Q1B.D
- new net BME_SDO: R3.2, U2.SDO/ADR
- new net CS: IC4.PA15, R22.1, R6.1
- new net CUT_ROPE: D12.C, Q1A.D
- new net D_PI: R51.2, U1.STAT_DIS
- new net D_RAD: R50.2, U3.STAT_DIS
- new net GPSRX2: IC4.PA10
- new net GPSTX2: IC4.PA9
- new net K_PI: IC4.PA5, R48.1, U1.INPUT
- new net K_RAD: IC4.PA3, R49.1, U3.INPUT
- new net L1: OK1A.A, R29.1
- new net L1+: R29.2
- new net L1-: OK1A.C
- new net L2: OK2A.A, R31.1
- new net L2+: R31.2
- new net L2-: OK2A.C
- new net L3: OK3A.A, R33.1
- new net L3+: R33.2
- new net L3-: OK3A.C
- new net L4: OK1B.A, R35.1
- new net L4+: R35.2
- new net L4-: OK1B.C
- new net L5: OK2B.A, R37.1
- new net L5+: R37.2
- new net L5-: OK2B.C
- new net L6: OK3B.A, R39.1
- new net L6+: R39.2
- new net L6-: OK3B.C
- new net LED1: IC4.PB12, OK1A.COL, R21.1
- new net LED2: IC4.PB13, OK2A.COL, R30.1
- new net LED3: IC4.PB14, OK3A.COL, R32.1
- new net LED4: IC4.PB15, OK1B.COL, R34.1
- new net LED5: IC4.PA8, OK2B.COL, R36.1
- new net LED6: IC4.PA11, OK3B.COL, R38.1
- new net LS1: J2.GP24, R44.1, R46.2
- new net LS2: J2.GP25, R45.1, R47.2
- new net N$1: Q1A.G, R44.2
- new net N$2: Q1B.G, R45.2
- new net R_CS0: J2.CE0
- new net R_CS1: J2.CE1
- new net R_MISO: J2.MISO
- new net R_MOSI: J2.MOSI
- new net R_RX: IC4.PB6, J2.RXI, R43.1
- new net R_SCK: J2.SCLK
- new net R_SCL: J2.SCL, JP4.1
- new net R_SDA: J2.SDA, JP3.1
- new net R_TX: IC4.PB7, J2.TXO, R42.1
- new net TEMP: D6.C, IC4.PA0, J8.3
- new net VRAD: IC4.PA1, R40.1, R41.2
- net 3.3V: now also R21.2, R30.2, R32.2, R34.2, R36.2, R38.2, R42.2, R43.2, R48.2, R49.2, R5.2, R8.2, U2.!CS, U2.VDD, U2.VDDIO; no longer C27.1, IC3A.G1, IC3P.VCC, J2.2, J4.VCC, R21.1, R29.1
- net 5V: now also C28.1, U1.VCC
- net B_MISO: no longer J3.9, R3A.1
- net B_MOSI: no longer J3.2, R8.2
- net B_SCK: no longer J3.4, R5.2
- net GND: now also D12.A, D13.A, D6.A, J2.GND@14, J2.GND@20, J2.GND@25, J2.GND@6, J2.GND@9, OK1A.EMIT, OK1B.EMIT, OK2A.EMIT, OK2B.EMIT, OK3A.EMIT, OK3B.EMIT, Q1A.S, Q1B.S, R3.1, R41.1, R46.1, R47.1, R50.1, R51.1, U1.GND, U2.GND1, U2.GND2, U3.GND; no longer C31.2, C32.2, C33.2, D6.GND, IC3A.G2, IC3P.GND, IC9.GND, J10.2, J12.2, J2.1, J3.1, J3.5, J4.CD1, J4.CD2, J4.GND, J4.SHIELD@1, J4.SHIELD@3, J9.2
- net MISO: no longer IC9.AL_H, J4.DO, R3A.2
- net MOSI: no longer J4.DI, R8.1
- net SCK: no longer IC9.SDA, J4.SCK, R5.1
- net SCL: now also JP4.2, R5.1, U2.SCK/SCL; no longer J2.4, R21.2
- net SDA: now also JP3.2, R8.1, U2.SDI/SDA; no longer J2.3, R29.2
- net VDIV: now also IC4.PA2; no longer IC4.PA3
- net VS: no longer C29.1, C31.1, C32.1, C33.1, D6.VCC, IC9.VDD, J10.1, J12.1, J3.10, J3.8, J9.1
Other:
- note added: "828-1063-1-ND"
- note added: "Alternative: STM32L433CCT6 497-16579-ND"
- note added: "L1: CVH252009-2R2MCT-ND C19-C20: 490-5523-1-ND C21: 493-10772-1-ND D1, D12, D13: CDSOD323-T15SCT-ND D2, D4-D10: DESD5V0U1BA-7DICT-ND"
- note added: "Raspberry Pi has I2C pull-up resistors"
- note removed: "HOUSING: 455-1151-ND CRIMP: 455-1127-1-ND SIDE: 455-1727-ND"
- note removed: "L1: CVH252009-2R2MCT-ND C19-C20: 490-5523-1-ND C21: 493-10772-1-ND D1: ESD12VD3-TPMSCT-ND D2, D5, D7-D9: DESD5V0U1BA-7DICT-ND"
- note removed: "NC"
- note removed: "YC164J-100CT-ND"
- note removed: "YC164J-10KCT-ND"
- moved on the sheet: C13, C16, C23, C24, C27, C28, C29, C30, C34, C35, C36, D10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

Commit message: Add Phoenix telemetry PCB
Parts:
- removed C15, C27, C35: 1u, SparkFun-Passives:CAP0805
- removed C17, C30: 0.1u, SparkFun-Passives:CAP0805
- removed IC1: COPERNICUSSMD, SparkFun-RF:COPERNICUSSMD
- removed J1: I2C1, SparkFun-Connectors:I2C_STANDARD_NO_SILK
- removed J13: LORA, HAB:1X08
- removed J5: BAT, SparkFun-Connectors:M02PTH
- removed J7: SMA_EDGE, SparkFun-Connectors:SMA_EDGE
- removed J8: TEMP_E, SparkFun-Connectors:M03JST-PTH
- removed JP1: GND, SparkFun-Passives:JUMPER-PAD-2-NC_BY_TRACE
- removed OK1, OK2, OK3: LTV826S, optocoupler:LTV826S
- removed R10\, R40: 430K, SparkFun-Passives:RESISTOR0805-RES
- removed R2: 10K, SparkFun-Passives:RESISTOR-ARRAY0603-ARV
- removed R24, R42: 10K, SparkFun-Passives:RESISTOR0805-RES
- removed R31, R33, R34, R35, R36, R37, R38, R39: 4.7K, SparkFun-Passives:RESISTOR0805-RES
- removed R41: 100K, SparkFun-Passives:RESISTOR0805-RES
- added D11: 5.6V, SparkFun-DiscreteSemi:DIODE-ZENER5.6V
- added D15: 15V, SparkFun-DiscreteSemi:DIODE-ZENER5.6V
- added J3: POWER, HAB:1X10
- added J4: GPS2, SparkFun-Connectors:M06SMD-1MM
- added J9: IO, SparkFun-Connectors:M08X2
- added R56: 470K, SparkFun-Passives:RESISTOR0805-RES
- D12: value 15V -> 5.6V
- J2: value RASPBERRYPI-GPIOPTH -> RASPBERRYPI-GPIO; device SparkFun-Boards:RASPBERRYPI-GPIOPTH -> HAB:RASPBERRYPI-GPIO
- R10: value 470K -> 430K
- R21, R29, R30: value 4.7K -> 100
- R25, R4: value 10K -> 100
- R27: value 330k -> 330K
- R28: value 0 -> 100
- R32: value 4.7K -> DNP
- Y2: device SparkFun-FreqCtrl:CRYSTALSMD -> SparkFun-FreqCtrl:CRYSTALTXC-7A
- renumbered U1 to IC9, U2 to IC3, U3 to IC11
Connections:
- net N$1 renamed CRB
- net N$2 renamed ACB
- removed net 15V: C29.1, IC11.VCC, R40.2
- removed net AGND: IC1.GND@2, IC1.GND@3, J7.GND@0, J7.GND@1, J7.GND@2, J7.GND@3, JP1.1
- removed net GPSBOOT: IC1.BOOT, R4.1
- removed net L1+: R29.2
- removed net L1-: OK1A.C
- removed net L2+: R31.2
- removed net L2-: OK2A.C
- removed net L3+: R33.2
- removed net L3-: OK3A.C
- removed net L4: OK1B.A, R35.1
- removed net L4+: R35.2
- removed net L4-: OK1B.C
- removed net L5: OK2B.A, R37.1
- removed net L5+: R37.2
- removed net L5-: OK2B.C
- removed net L6: OK3B.A, R39.1
- removed net L6+: R39.2
- removed net L6-: OK3B.C
- removed net LED4: IC4.PB15, OK1B.COL, R34.1
- removed net LED5: IC4.PA8, OK2B.COL, R36.1
- removed net LED6: IC4.PA11, OK3B.COL, R38.1
- removed net LP-: IC7B.-IN, R28.1
- removed net PPS: IC1.PPS
- removed net RF_GPS: IC1.RFIN, J7.SIGNAL
- removed net RXA: IC1.RXD-A, R2B.2
- removed net TXA: IC1.TXD-A, R2C.2
- removed net VRAD: IC4.PA1, R40.1, R41.2
- removed net XRESET: IC1.XRESET, R24.2
- removed net XSTBY: IC1.XSTANDBY, IC4.PB2, R25.2
- new net +9V: J3.6, J3.7, J3.8
- new net 3V_PI: J2.3.3V@1
- new net 3V_PI2: J2.3.3V@17
- net 15V_OUT: now also J3.4
- net 3.3V: now also D12.C, J9.7, J9.8; no longer C11.1, C12.1, C15.1, C16.1, D10.C, IC1.VCC, IC3.!CS, IC3.VDD, IC3.VDDIO, J1.2, J13.7, J13.8, R21.2, R24.1, R25.1, R2B.1, R2C.1, R2D.1, R30.2, R34.2, R36.2, R38.2, R4.2, R42.2
- net 5V: now also J4.2, R10.2; no longer C17.1, R10\.2
- net 5V_PI: no longer C27.1
- net A-: now also R56.2; no longer R10.2
- net ALT_CTRL: now also J3.9
- net B_LORA: now also D10.C, J9.14; no longer J13.3
- net B_MISO: now also J9.10, R28.1; no longer J13.6
- net B_MOSI: now also J9.6, R25.1; no longer J13.2
- net B_SCK: now also J9.12, R4.1; no longer J13.4
- net CUT_ROPE: now also D15.C, J3.10; no longer D12.C
- net FB5: now also R10.1; no longer R10\.1
- net GND: now also D11.A, D15.A, J3.2, J3.3, J3.5, J4.1, J4.5, J9.15, J9.16, J9.9, R56.1; no longer C11.2, C12.2, C15.2, C17.2, C27.2, C30.2, C35.2, IC1.GND@1, IC1.GND@4, IC1.GND@5, IC1.GND@6, IC1.GND@7, IC1.GND@8, J1.1, J13.1, J13.5, J5.1, J8.2, JP1.2, OK1A.EMIT, OK1B.EMIT, OK2A.EMIT, OK2B.EMIT, OK3A.EMIT, OK3B.EMIT, R10.1, R41.1
- net GPSRX: no longer IC1.TXD-B, R2D.2
- net GPSRX2: now also J4.4
- net GPSTX: no longer IC1.RXD-B
- net GPSTX2: now also J4.3
- net K_PI: now also IC4.PA0; no longer IC4.PA5
- net K_RAD: now also IC4.PA8; no longer IC4.PA3
- net L1: now also J9.2, R21.1; no longer OK1A.A, R29.1
- net L2: now also J9.1, R29.1; no longer OK2A.A, R31.1
- net L3: now also J9.4, R30.1; no longer OK3A.A, R33.1
- net LED1: now also IC4.PA3, R21.2; no longer IC4.PB12, OK1A.COL, R21.1
- net LED2: now also IC4.PA2, R29.2; no longer IC4.PB13, OK2A.COL, R30.1
- net LED3: now also IC4.PA1, R30.2; no longer IC4.PB14, OK3A.COL, R32.1
- net LS1: now also J2.GP25; no longer J2.GP24
- net LS2: now also J2.GP24; no longer J2.GP25
- net MISO: now also R28.2
- net MOSI: now also R25.2
- net R_TX: no longer R42.1
- net SCK: now also R4.2
- net SCL: now also J9.5; no longer J1.4
- net SDA: now also J9.3; no longer J1.3
- net TEMP: now also IC4.PB15, J9.13, R32.1; no longer IC4.PA0, J8.3
- net TXD: now also IC7B.-IN; no longer R28.2
- net VBAT: now also C29.1, IC11.VCC, J3.1; no longer J5.2
- net VDIV: now also IC4.PA5; no longer IC4.PA2
- net VS: now also C16.1, D11.C, IC3.!CS, IC3.VDD, IC3.VDDIO, J9.11; no longer C30.1, C35.1, J8.1
Other:
- note added: "887-1448-1-ND"
- note added: "L1: CVH252009-2R2MCT-ND C19, C20, C31: 490-5523-1-ND C21: 493-10772-1-ND D1, D13-D15: CDSOD323-T15SCT-ND D2, D4-D12: DESD5V0U1BA-7DICT-ND"
- note removed: "887-1233-ND"
- note removed: "L1: CVH252009-2R2MCT-ND C19-C20: 490-5523-1-ND C21: 493-10772-1-ND D1, D12, D13: CDSOD323-T15SCT-ND D2, D4-D10: DESD5V0U1BA-7DICT-ND"
- note removed: "PLUG: 455-1710-ND"
- moved on the sheet: C11, C12, C22, C6, C7, C8, C9, D10, D12, D4, D5, D6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

Commit message: Add GPS1 connector to Phoenix board
Parts:
- removed FRAME3: FRAME-LETTERNO_PACKAGE, SparkFun-Aesthetics:FRAME-LETTERNO_PACKAGE
- added J1: GPS1, SparkFun-Connectors:M04PTH
- R56: value 470K -> 430K
Connections:
- net 3.3V: now also C11.1, C12.1
- net GND: now also C11.2, C12.2, J1.1
- net GPSRX: now also J1.3
- net GPSTX: now also J1.2
- net VS: now also J1.4
Other:
- note added: "L1: CVH252009-2R2MCT-ND C19, C20, C31: 1276-2890-1-ND C21: 493-10772-1-ND D1, D13-D15: CDSOD323-T15SCT-ND D2, D4-D12: DESD5V0U1BA-7DICT-ND"
- note removed: "L1: CVH252009-2R2MCT-ND C19, C20, C31: 490-5523-1-ND C21: 493-10772-1-ND D1, D13-D15: CDSOD323-T15SCT-ND D2, D4-D12: DESD5V0U1BA-7DICT-ND"
- moved on the sheet: C11, C12, C28, C29, IC11, IC9, R48, R49, R50, R51

Commit message: Rotate and reroute Phoenix board, much cleaner!
Parts:
- removed J11: DNP, SparkFun-Connectors:M06LOCK
- added J5: DNP, SparkFun-Connectors:M04LOCK
- C21: device SparkFun-Passives:CAP_POLPTH2 -> SparkFun-Passives:CAP_POLE
Connections:
- net !RST!: now also J5.4; no longer J11.5
- net 3.3V: now also J1.4; no longer J11.1
- net B_LORA: now also J9.6; no longer J9.14
- net B_MISO: now also J9.12; no longer J9.10
- net B_MOSI: now also J9.14; no longer J9.6
- net B_SCK: now also J9.10; no longer J9.12
- net GND: now also J1.3, J5.2; no longer J1.1, J11.3
- net GPSRX: now also J1.2; no longer J1.3
- net GPSTX: now also J1.1; no longer J1.2
- net SWCLK: now also J5.1; no longer J11.2
- net SWDIO: now also J5.3; no longer J11.4
- net VS: no longer J1.4
Changed lines of the file:
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@@
 <part name="C19" library="SparkFun-Passives" deviceset="CAP" device="0805" value="10u"/>
 <part name="R9" library="SparkFun-Passives" deviceset="RESISTOR" device="0805-RES" value="10K"/>
-<part name="C21" library="SparkFun-Passives" deviceset="CAP_POL" device="PTH2" value="100u"/>
+<part name="C21" library="SparkFun-Passives" deviceset="CAP_POL" device="E" value="100u"/>
 <part name="GND20" library="SparkFun-Aesthetics" deviceset="GND" device=""/>
 <part name="GND21" library="SparkFun-Aesthetics" deviceset="GND" device=""/>
@@
 <part name="R20" library="SparkFun-Passives" deviceset="RESISTOR" device="0805-RES" value="100K"/>
 <part name="GND32" library="SparkFun-Aesthetics" deviceset="GND" device=""/>
-<part name="J11" library="SparkFun-Connectors" deviceset="M06" device="LOCK" value="DNP"/>
 <part name="GND37" library="SparkFun-Aesthetics" deviceset="GND" device=""/>
-<part name="SUPPLY29" library="SparkFun-Aesthetics" deviceset="3.3V" device=""/>
 <part name="JP2" library="SparkFun-Passives" deviceset="JUMPER-PAD-2-NC_BY_TRACE" device="" value="GND"/>
 <part name="GND42" library="SparkFun-Aesthetics" deviceset="GND" device=""/>
@@
 <part name="GND9" library="SparkFun-Aesthetics" deviceset="GND" device=""/>
 <part name="J1" library="SparkFun-Connectors" deviceset="M04" device="PTH" value="GPS1"/>
+<part name="SUPPLY8" library="SparkFun-Aesthetics" deviceset="3.3V" device=""/>
+<part name="J5" library="SparkFun-Connectors" deviceset="M04" device="LOCK" value="DNP"/>
 </parts>
 <sheets>
@@
 <instance part="R20" gate="G$1" x="416.56" y="157.48" rot="R90"/>
 <instance part="GND32" gate="1" x="416.56" y="147.32"/>
-<instance part="J11" gate="G$1" x="71.12" y="17.78" rot="R180"/>
 <instance part="GND37" gate="1" x="63.5" y="5.08"/>
-<instance part="SUPPLY29" gate="G$1" x="63.5" y="22.86"/>
 <instance part="JP2" gate="G$1" x="134.62" y="33.02"/>
 <instance part="GND42" gate="1" x="233.68" y="50.8"/>
@@
 <instance part="GND9" gate="1" x="284.48" y="10.16"/>
 <instance part="J1" gate="G$1" x="276.86" y="17.78"/>
+<instance part="SUPPLY8" gate="G$1" x="284.48" y="25.4"/>
+<instance part="J5" gate="G$1" x="71.12" y="17.78" rot="R180"/>
 </instances>
 <busses>
@@
 </segment>
 <segment>
-<pinref part="J11" gate="G$1" pin="3"/>
 <pinref part="GND37" gate="1" pin="GND"/>
 <wire x1="66.04" y1="17.78" x2="63.5" y2="17.78" width="0.1524" layer="91"/>
 <wire x1="63.5" y1="17.78" x2="63.5" y2="7.62" width="0.1524" layer="91"/>
+<pinref part="J5" gate="G$1" pin="2"/>
 </segment>
 <segment>
@@
 </segment>
 <segment>
-<pinref part="J1" gate="G$1" pin="1"/>
 <pinref part="GND9" gate="1" pin="GND"/>
-<wire x1="281.94" y1="15.24" x2="284.48" y2="15.24" width="0.1524" layer="91"/>
-<wire x1="284.48" y1="15.24" x2="284.48" y2="12.7" width="0.1524" layer="91"/>
+<wire x1="284.48" y1="12.7" x2="284.48" y2="20.32" width="0.1524" layer="91"/>
+<pinref part="J1" gate="G$1" pin="3"/>
+<wire x1="284.48" y1="20.32" x2="281.94" y2="20.32" width="0.1524" layer="91"/>
 </segment>
 </net>
@@
 <pinref part="R7" gate="G$1" pin="2"/>
 <wire x1="101.6" y1="124.46" x2="101.6" y2="121.92" width="0.1524" layer="91"/>
-</segment>
-<segment>
-<pinref part="SUPPLY29" gate="G$1" pin="3.3V"/>
-<pinref part="J11" gate="G$1" pin="1"/>
-<wire x1="63.5" y1="22.86" x2="66.04" y2="22.86" width="0.1524" layer="91"/>
 </segment>
 <segment>
@@
 <junction x="398.78" y="20.32"/>
 </segment>
+<segment>
+<pinref part="SUPPLY8" gate="G$1" pin="3.3V"/>
+<wire x1="284.48" y1="25.4" x2="284.48" y2="22.86" width="0.1524" layer="91"/>
+<pinref part="J1" gate="G$1" pin="4"/>
+<wire x1="284.48" y1="22.86" x2="281.94" y2="22.86" width="0.1524" layer="91"/>
+</segment>
 </net>
 <net name="VDDA" class="0">
@@
 </segment>
 <segment>
-<pinref part="J11" gate="G$1" pin="5"/>
 <wire x1="53.34" y1="12.7" x2="66.04" y2="12.7" width="0.1524" layer="91"/>
 <label x="53.34" y="12.7" size="1.778" layer="95"/>
+<pinref part="J5" gate="G$1" pin="4"/>
 </segment>
 </net>
@@
 </segment>
 <segment>
-<pinref part="J11" gate="G$1" pin="2"/>
 <wire x1="53.34" y1="20.32" x2="66.04" y2="20.32" width="0.1524" layer="91"/>
 <label x="53.34" y="20.32" size="1.778" layer="95"/>
+<pinref part="J5" gate="G$1" pin="1"/>
 </segment>
 </net>
@@
 </segment>
 <segment>
-<pinref part="J11" gate="G$1" pin="4"/>
 <wire x1="53.34" y1="15.24" x2="66.04" y2="15.24" width="0.1524" layer="91"/>
 <label x="53.34" y="15.24" size="1.778" layer="95"/>
+<pinref part="J5" gate="G$1" pin="3"/>
 </segment>
 </net>
@@
 </segment>
 <segment>
-<wire x1="292.1" y1="17.78" x2="281.94" y2="17.78" width="0.1524" layer="91"/>
-<label x="289.56" y="17.78" size="1.778" layer="95"/>
-<pinref part="J1" gate="G$1" pin="2"/>
+<pinref part="J1" gate="G$1" pin="1"/>
+<wire x1="289.56" y1="15.24" x2="281.94" y2="15.24" width="0.1524" layer="91"/>
+<label x="287.02" y="15.24" size="1.778" layer="95"/>
 </segment>
 </net>
@@
 </segment>
 <segment>
-<wire x1="292.1" y1="20.32" x2="281.94" y2="20.32" width="0.1524" layer="91"/>
-<label x="289.56" y="20.32" size="1.778" layer="95"/>
-<pinref part="J1" gate="G$1" pin="3"/>
+<wire x1="289.56" y1="17.78" x2="281.94" y2="17.78" width="0.1524" layer="91"/>
+<label x="287.02" y="17.78" size="1.778" layer="95"/>
+<pinref part="J1" gate="G$1" pin="2"/>
 </segment>
 </net>
@@
 </segment>
 <segment>
+<pinref part="J9" gate="G$1" pin="12"/>
+<wire x1="231.14" y1="60.96" x2="238.76" y2="60.96" width="0.1524" layer="91"/>
+<label x="236.22" y="60.96" size="1.778" layer="95"/>
+</segment>
+</net>
+<net name="B_MOSI" class="0">
+<segment>
+<pinref part="D9" gate="G$1" pin="C"/>
+<wire x1="480.06" y1="53.34" x2="480.06" y2="58.42" width="0.1524" layer="91"/>
+<label x="480.06" y="55.88" size="1.778" layer="95" rot="R90"/>
+</segment>
+<segment>
+<pinref part="R25" gate="G$1" pin="1"/>
+<wire x1="378.46" y1="129.54" x2="373.38" y2="129.54" width="0.1524" layer="91"/>
+<label x="375.92" y="129.54" size="1.778" layer="95"/>
+</segment>
+<segment>
+<wire x1="238.76" y1="58.42" x2="231.14" y2="58.42" width="0.1524" layer="91"/>
+<label x="236.22" y="58.42" size="1.778" layer="95"/>
+<pinref part="J9" gate="G$1" pin="14"/>
+</segment>
+</net>
+<net name="B_SCK" class="0">
+<segment>
+<pinref part="D8" gate="G$1" pin="C"/>
+<wire x1="467.36" y1="53.34" x2="467.36" y2="58.42" width="0.1524" layer="91"/>
+<label x="467.36" y="55.88" size="1.778" layer="95" rot="R90"/>
+</segment>
+<segment>
+<pinref part="R4" gate="G$1" pin="1"/>
+<wire x1="378.46" y1="137.16" x2="373.38" y2="137.16" width="0.1524" layer="91"/>
+<label x="375.92" y="137.16" size="1.778" layer="95"/>
+</segment>
+<segment>
 <wire x1="238.76" y1="63.5" x2="231.14" y2="63.5" width="0.1524" layer="91"/>
 <label x="236.22" y="63.5" size="1.778" layer="95"/>
 <pinref part="J9" gate="G$1" pin="10"/>
-</segment>
-</net>
-<net name="B_MOSI" class="0">
-<segment>
-<pinref part="D9" gate="G$1" pin="C"/>
-<wire x1="480.06" y1="53.34" x2="480.06" y2="58.42" width="0.1524" layer="91"/>
-<label x="480.06" y="55.88" size="1.778" layer="95" rot="R90"/>
-</segment>
-<segment>
-<pinref part="R25" gate="G$1" pin="1"/>
-<wire x1="378.46" y1="129.54" x2="373.38" y2="129.54" width="0.1524" layer="91"/>
-<label x="375.92" y="129.54" size="1.778" layer="95"/>
-</segment>
-<segment>
-<wire x1="238.76" y1="68.58" x2="231.14" y2="68.58" width="0.1524" layer="91"/>
-<label x="236.22" y="68.58" size="1.778" layer="95"/>
-<pinref part="J9" gate="G$1" pin="6"/>
-</segment>
-</net>
-<net name="B_SCK" class="0">
-<segment>
-<pinref part="D8" gate="G$1" pin="C"/>
-<wire x1="467.36" y1="53.34" x2="467.36" y2="58.42" width="0.1524" layer="91"/>
-<label x="467.36" y="55.88" size="1.778" layer="95" rot="R90"/>
-</segment>
-<segment>
-<pinref part="R4" gate="G$1" pin="1"/>
-<wire x1="378.46" y1="137.16" x2="373.38" y2="137.16" width="0.1524" layer="91"/>
-<label x="375.92" y="137.16" size="1.778" layer="95"/>
-</segment>
-<segment>
-<pinref part="J9" gate="G$1" pin="12"/>
-<wire x1="231.14" y1="60.96" x2="238.76" y2="60.96" width="0.1524" layer="91"/>
-<label x="236.22" y="60.96" size="1.778" layer="95"/>
 </segment>
 </net>
@@
 <label x="203.2" y="60.96" size="1.778" layer="95"/>
 </segment>
-<segment>
-<pinref part="J1" gate="G$1" pin="4"/>
-<wire x1="281.94" y1="22.86" x2="292.1" y2="22.86" width="0.1524" layer="91"/>
-<label x="289.56" y="22.86" size="1.778" layer="95"/>
-</segment>
 </net>
 <net name="LP1" class="0">
@@
 </segment>
 <segment>
-<wire x1="238.76" y1="58.42" x2="231.14" y2="58.42" width="0.1524" layer="91"/>
-<label x="236.22" y="58.42" size="1.778" layer="95"/>
-<pinref part="J9" gate="G$1" pin="14"/>
-</segment>
-</net>
+<wire x1="238.76" y1="68.58" x2="231.14" y2="68.58" width="0.1524" layer="91"/>
+<label x="236.22" y="68.58" size="1.778" layer="95"/>
+<pinref part="J9" gate="G$1" pin="6"/>
+</segment>
+</net>
