File: hardware/telemetry-r2.sch (EAGLE design)
At the start: 110 parts, among them IC1 COPERNICUSSMD, IC10 TPS70933, IC2 TPS70933, IC3 74HC137, IC4 STM32L073CZT6, IC5 TPS62160, IC6 HX1, IC7 LMP7702, IC8 ADXL345, IC9 HIH9131, J1 I2C1, J10 TEMP_BAT, J11 DNP, J12 PHOTO_GP2, J13 LORA, J2 I2C2, J3 BOTTOM, J4 USD-SOCKET, J5 BAT, J6 SMA_EDGE, J7 SMA_EDGE, J8 TEMP_GPS, J9 PHOTO_GP4, Y1 32768, Y2 8M

Commit message: Start work on revised telemetry MCU using lessons learned from second HAB launch
Parts:
- removed C15, C35: 1u, SparkFun-Passives:CAP0805
- removed C17, C27, C29, C30, C31, C32, C33: 0.1u, SparkFun-Passives:CAP0805
- removed D10: 5.6V, SparkFun-DiscreteSemi:DIODE-ZENER5.6V
- removed J10: TEMP_BAT, SparkFun-Connectors:M03JST-PTH
- removed J11: DNP, SparkFun-Connectors:M06LOCK
- removed J12: PHOTO_GP2, SparkFun-Connectors:M03JST-PTH
- removed J13: LORA, HAB:1X08
- removed J7: SMA_EDGE, SparkFun-Connectors:SMA_EDGE
- removed J8: TEMP_GPS, SparkFun-Connectors:M03JST-PTH
- removed J9: PHOTO_GP4, SparkFun-Connectors:M03JST-PTH
- removed JP1: GND, SparkFun-Passives:JUMPER-PAD-2-NC_BY_TRACE
- removed R10\: 430K, SparkFun-Passives:RESISTOR0805-RES
- removed R21, R29: 4.7K, SparkFun-Passives:RESISTOR0805-RES
- removed R22: 100, SparkFun-Passives:RESISTOR0805-RES
- removed R24, R25, R28: 10K, SparkFun-Passives:RESISTOR0805-RES
- added D11, D12: 5.6V, SparkFun-DiscreteSemi:DIODE-ZENER5.6V
- added JP3: SDA, SparkFun-Jumpers:JUMPER-SMT_2_NO_SILK
- added JP4: SCL, SparkFun-Jumpers:JUMPER-SMT_2_NO_SILK
- added R32: 4.7K, SparkFun-Passives:RESISTOR0805-RES
- added R43, R48, R51: 10K, SparkFun-Passives:RESISTOR0805-RES
- added R56: 430K, SparkFun-Passives:RESISTOR0805-RES
- C13: value 1u -> 10u
- C21: device SparkFun-Passives:CAP_POLPTH2 -> SparkFun-Passives:CAP_POLE
- D1: value 12V -> 15V
- D6: value CM1213A -> 5.6V; device HAB:CM1213A -> SparkFun-DiscreteSemi:DIODE-ZENER5.6V
- IC1: value COPERNICUSSMD -> RA02; device SparkFun-RF:COPERNICUSSMD -> HAB:RA02
- IC3: value 74HC137 -> BME280; device HAB:74LS137PW -> BME280ComponentLibrary:BME280
- IC4: value STM32L073CZT6 -> STM32L052C8T6
- IC9: value HIH9131 -> VN5160S-E; device SparkFun-AnalogIC:HIH6131 -> HAB:VN5160S-E
- J1: value I2C1 -> GPS1; device SparkFun-Connectors:I2C_STANDARD_NO_SILK -> SparkFun-Connectors:M04PTH
- J2: value I2C2 -> RASPBERRYPI-GPIO; device SparkFun-Connectors:I2C_STANDARD_NO_SILK -> HAB:RASPBERRYPI-GPIO
- J3: value BOTTOM -> POWER; device SparkFun-Connectors:M102MM -> HAB:1X02
- J4: value USD-SOCKET -> GPS2; device SparkFun-Connectors:USD-SOCKET -> SparkFun-Connectors:M06SMD-1MM
- J5: value BAT -> DNP; device SparkFun-Connectors:M02PTH -> SparkFun-Connectors:M04LOCK
- R10, R19: value 470K -> 430K
- R2: device SparkFun-Passives:RESISTOR-ARRAY0603-ARV -> SparkFun-Passives:RESISTOR0805-RES
- R20: value 180K -> 100K
- R27: value 330k -> 330K
- R3: value 100 -> 10K; device SparkFun-Passives:RESISTOR-ARRAY0603-ARV -> SparkFun-Passives:RESISTOR0805-RES
- R5, R8: value 100 -> 3.3K
- Y2: device SparkFun-FreqCtrl:CRYSTALSMD -> SparkFun-FreqCtrl:CRYSTALTXC-7A
Connections:
- removed net +9V: C18.1, C21.+, D1.C, IC5.EN, IC5.VIN, J5.2, R19.2
- removed net AGND: IC1.GND@2, IC1.GND@3, J7.GND@0, J7.GND@1, J7.GND@2, J7.GND@3, JP1.1
- removed net AL_L: IC9.AL_L
- removed net B_CSADC: J3.7, R3B.1
- removed net B_CSHUM: J3.3, R3D.1
- removed net B_CSPRS: J3.6, R3C.1
- removed net B_LORA: J13.3, R22.2
- removed net B_MISO: D4.C, J13.6, J3.9, R3A.1
- removed net B_MOSI: D9.C, J13.2, J3.2, R8.2
- removed net B_SCK: D8.C, J13.4, J3.4, R5.2
- removed net CSA0: IC3A.A, IC4.PB7
- removed net CSA1: IC3A.B, IC4.PB6
- removed net CSA2: IC3A.C, IC4.PB12
- removed net CSADC: IC3A.Y5, R3B.2
- removed net CSBHUM: IC3A.Y3, R3D.2
- removed net CSHUM: IC3A.Y2, IC9.SCL
- removed net CSLAT: IC3A.GL, IC4.PA15, R6.1
- removed net CSLORA: IC3A.Y1, R22.1
- removed net CSPRS: IC3A.Y4, R3C.2
- removed net CSSD: IC3A.Y0, J4.CS
- removed net D+: IC4.PA12
- removed net D-: IC4.PA11
- removed net GPSBOOT: IC1.BOOT, R4.1
- removed net LP-: IC7B.-IN, R28.1
- removed net MCO: IC4.PA8
- removed net PHOTO_GP2: D6.CH2, IC4.PA5, J12.3
- removed net PHOTO_GP4: D6.CH1, IC4.PA2, J9.3
- removed net PPS: IC1.PPS
- removed net RF_GPS: IC1.RFIN, J7.SIGNAL
- removed net RXA: IC1.RXD-A, R2B.2
- removed net TEMPB: D6.CH4, IC4.PA1, J10.3
- removed net TEMPG: D6.CH3, IC4.PA0, J8.3
- removed net TXA: IC1.TXD-A, R2C.2
- removed net USIN: IC4.PB14
- removed net USOUT: IC4.PB15
- removed net USRES: IC4.PB13
- removed net VCORE: C28.1, IC9.VCORE
- removed net XRESET: IC1.XRESET, R24.2
- removed net XSTBY: IC1.XSTANDBY, IC4.PB2, R25.2
- new net !LORA_IRQ!: IC1.DIO0
- new net !LORA_RST!: IC1.!RESET!, R2.1
- new net 3V_PI: J2.3.3V@1
- new net 3V_PI2: J2.3.3V@17
- new net 5V_PI: IC9.OUTPUT, J2.5V@2, J2.5V@4
- new net BME_SDO: IC3.SDO/ADR, R3.2
- new net D_PI: IC9.STAT_DIS, R51.2
- new net GPSRX2: IC4.PA10, J4.4
- new net GPSTX2: IC4.PA9, J4.3
- new net K_PI: IC4.PA0, IC9.INPUT, R48.1
- new net LCS: IC1.!SS!, IC4.PB7, R4.1
- new net R_CS0: J2.CE0
- new net R_CS1: J2.CE1
- new net R_MISO: J2.MISO
- new net R_MOSI: J2.MOSI
- new net R_RX: IC4.PA3, J2.RXI, R43.1
- new net R_SCK: J2.SCLK
- new net R_SCL: J2.SCL, JP4.1
- new net R_SDA: J2.SDA, JP3.1
- new net R_TX: IC4.PA2, J2.TXO
- new net SDCS: IC4.PA15, R6.1
- new net TEMP: D6.C, IC4.PB15, R32.1
- new net U_RX: IC4.PB6
- new net VBAT: C18.1, C21.+, D1.C, IC5.EN, IC5.VIN, J3.1, R19.2
- net !RST!: now also J5.4; no longer J11.5
- net 3.3V: now also D12.C, J1.4, R2.2, R32.2, R43.2, R48.2, R5.2, R8.2; no longer C15.1, C16.1, C27.1, D10.C, IC3A.G1, IC3P.VCC, J1.2, J11.1, J13.7, J13.8, J2.2, J4.VCC, R21.1, R24.1, R25.1, R26.2, R29.1, R2B.1, R2C.1, R2D.1
- net 5V: now also C28.1, IC9.VCC, J4.2, R10.2; no longer C17.1, R10\.2
- net A-: now also R56.2; no longer R10.2
- net FB5: now also R10.1; no longer R10\.1
- net GND: now also D11.A, D12.A, D6.A, IC1.GND, IC2.NC/FB, IC3.GND1, IC3.GND2, J1.3, J2.GND@14, J2.GND@20, J2.GND@25, J2.GND@6, J2.GND@9, J3.2, J4.1, J4.5, J5.2, R26.2, R3.1, R51.1, R56.1; no longer C15.2, C17.2, C27.2, C29.2, C30.2, C31.2, C32.2, C33.2, C35.2, D10.A, D6.GND, IC1.GND@1, IC1.GND@4, IC1.GND@5, IC1.GND@6, IC1.GND@7, IC1.GND@8, IC3A.G2, IC3P.GND, J1.1, J10.2, J11.3, J12.2, J13.1, J13.5, J2.1, J3.1, J3.5, J4.CD1, J4.CD2, J4.GND, J4.SHIELD@1, J4.SHIELD@3, J5.1, J8.2, J9.2, JP1.2, R10.1
- net GPSRX: now also J1.2; no longer IC1.TXD-B, R2D.2
- net GPSTX: now also J1.1; no longer IC1.RXD-B
- net MISO: now also D4.C, IC1.MISO; no longer IC9.AL_H, J4.DO, R3A.2
- net MOSI: now also D9.C, IC1.MOSI; no longer J4.DI, R8.1
- net SCK: now also D8.C, IC1.SCK; no longer IC9.SDA, J4.SCK, R5.1
- net SCL: now also IC3.SCK/SCL, JP4.2, R5.1; no longer J1.4, J2.4, R21.2
- net SDA: now also IC3.SDI/SDA, JP3.2, R8.1; no longer J1.3, J2.3, R29.2
- net SWCLK: now also J5.1; no longer J11.2
- net SWDIO: now also J5.3; no longer J11.4
- net TXD: now also IC7B.-IN; no longer R28.2
- net VDIV: now also IC4.PA5; no longer IC4.PA3
- net VS: now also C16.1, D11.C, IC3.!CS, IC3.VDD, IC3.VDDIO; no longer C29.1, C30.1, C31.1, C32.1, C33.1, C35.1, D6.VCC, IC9.VDD, J10.1, J12.1, J3.10, J3.8, J8.1, J9.1
Other:
- note added: "828-1063-1-ND"
- note added: "887-1448-1-ND"
- note added: "A121350-ND"
- note added: "Alternative: STM32L433CCT6 497-16579-ND"
- note added: "L1: CVH252009-2R2MCT-ND C19, C20, C31: 1276-2890-1-ND C21: 493-10772-1-ND D1, D13-D15: CDSOD323-T15SCT-ND D2, D4-D12: DESD5V0U1BA-7DICT-ND"
- note removed: "887-1233-ND"
- note removed: "HOUSING: 455-1151-ND CRIMP: 455-1127-1-ND SIDE: 455-1727-ND"
- note removed: "L1: CVH252009-2R2MCT-ND C19-C20: 490-5523-1-ND C21: 493-10772-1-ND D1: ESD12VD3-TPMSCT-ND D2, D5, D7-D9: DESD5V0U1BA-7DICT-ND"
- note removed: "NC"
- note removed: "PLUG: 455-1710-ND"
- note removed: "YC164J-100CT-ND"
- note removed: "YC164J-10KCT-ND"
- moved on the sheet: C11, C12, C13, C16, C22, C23, C24, C28, C34, C36, C6, C7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
