File: hardware/tmod-pi.brd (EAGLE design)
At the start: 65 x 56 mm, 25 parts, among them J1 RASPBERRYPI-40-PIN-GPIO_PTH, J2 HAB-EXP, J3 GROVE, J4 SMA_EDGE, U1 DNP (74AHC1G125), U2 DNP (PCA9306), U3 DNP (74AHC1G125), U4 RA01

Commit message: Continued work on the Pi-style application board
Routing:
- net LCS: track 0.00 -> 32.0 mm
- net PI_RX: track 1.76 -> 23.9 mm, vias 0 -> 1
- net 3V_PI: track 4.38 -> 24.6 mm, vias 0 -> 3
- net 3.3V: track 16.0 -> 30.2 mm, vias 0 -> 2
- net PI_TX: track 6.32 -> 17.2 mm
- net PI_SCL: track 15.5 -> 16.2 mm
- net P_SCL: track 10.0 -> 10.5 mm
- added copper zone on layer 1, net 3V_PI
Changed lines of the file:
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@@
 <contactref element="J4" pad="GND@1"/>
 <contactref element="J4" pad="GND@0"/>
-<via x="15.875" y="42.926" extent="1-16" drill="0.5"/>
+<via x="16.51" y="42.926" extent="1-16" drill="0.5"/>
 <contactref element="C5" pad="2"/>
+<via x="24.13" y="42.926" extent="1-16" drill="0.5"/>
+<via x="29.21" y="41.021" extent="1-16" drill="0.5"/>
 </signal>
 <signal name="3.3V">
@@
 <wire x1="40.815" y1="8.51" x2="40.815" y2="5.275" width="0.6096" layer="1"/>
 <wire x1="40.815" y1="5.275" x2="41.645" y2="4.445" width="0.6096" layer="1"/>
+<wire x1="25.03" y1="40.005" x2="26.035" y2="40.005" width="0.4064" layer="1"/>
+<via x="26.035" y="40.005" extent="1-16" drill="0.5"/>
+<wire x1="26.035" y1="40.005" x2="17.78" y2="40.005" width="0.4064" layer="16"/>
+<wire x1="17.78" y1="40.005" x2="15.24" y2="42.545" width="0.4064" layer="16"/>
+<wire x1="14.065" y1="43.0192" x2="14.7658" y2="43.0192" width="0.3048" layer="1"/>
+<wire x1="14.7658" y1="43.0192" x2="15.24" y2="42.545" width="0.3048" layer="1"/>
+<via x="15.24" y="42.545" extent="1-16" drill="0.5"/>
 <wire x1="40.815" y1="8.51" x2="62.865" y2="36.83" width="0" layer="19" extent="1-1"/>
-<wire x1="25.03" y1="40.005" x2="40.815" y2="8.51" width="0" layer="19" extent="1-1"/>
-<wire x1="14.065" y1="43.0192" x2="25.08" y2="41.8799" width="0" layer="19" extent="1-1"/>
+<wire x1="26.035" y1="40.005" x2="40.815" y2="8.51" width="0" layer="19" extent="1-1"/>
 </signal>
 <signal name="5V">
@@
 <wire x1="23.495" y1="46.355" x2="21.59" y2="46.355" width="0.2032" layer="1"/>
 <wire x1="21.59" y1="46.355" x2="21.59" y2="44.08" width="0.2032" layer="1"/>
-<wire x1="21.59" y1="46.355" x2="15.99" y2="53.77" width="0" layer="19" extent="1-1"/>
+<wire x1="21.59" y1="46.355" x2="21.59" y2="47.625" width="0.2032" layer="1"/>
+<wire x1="21.59" y1="47.625" x2="19.685" y2="49.53" width="0.2032" layer="1"/>
+<wire x1="19.685" y1="49.53" x2="17.78" y2="49.53" width="0.2032" layer="1"/>
+<wire x1="17.78" y1="49.53" x2="17.272" y2="50.038" width="0.2032" layer="1"/>
+<wire x1="17.272" y1="50.038" x2="17.272" y2="52.488" width="0.2032" layer="1"/>
+<wire x1="17.272" y1="52.488" x2="15.99" y2="53.77" width="0.2032" layer="1"/>
 </signal>
 <signal name="PI_RX">
@@
 <wire x1="30.16" y1="41.9401" x2="31.3499" y2="41.9401" width="0.2032" layer="1"/>
 <wire x1="31.3499" y1="41.9401" x2="31.75" y2="41.54" width="0.2032" layer="1"/>
-<wire x1="30.16" y1="41.9401" x2="18.53" y2="53.77" width="0" layer="19" extent="1-1"/>
+<wire x1="30.16" y1="41.9401" x2="30.16" y2="42.225" width="0.2032" layer="1"/>
+<wire x1="30.16" y1="42.225" x2="31.75" y2="43.815" width="0.2032" layer="1"/>
+<wire x1="31.75" y1="43.815" x2="31.75" y2="45.72" width="0.2032" layer="1"/>
+<via x="31.75" y="45.72" extent="1-16" drill="0.5"/>
+<wire x1="31.75" y1="45.72" x2="28.575" y2="48.895" width="0.2032" layer="16"/>
+<wire x1="28.575" y1="48.895" x2="23.495" y2="48.895" width="0.2032" layer="16"/>
+<wire x1="23.495" y1="48.895" x2="22.352" y2="50.038" width="0.2032" layer="16"/>
+<wire x1="22.352" y1="50.038" x2="22.352" y2="51.943" width="0.2032" layer="16"/>
+<wire x1="22.352" y1="51.943" x2="21.717" y2="52.578" width="0.2032" layer="16"/>
+<wire x1="21.717" y1="52.578" x2="19.722" y2="52.578" width="0.2032" layer="16"/>
+<wire x1="19.722" y1="52.578" x2="18.53" y2="53.77" width="0.2032" layer="16"/>
 </signal>
 <signal name="UART_EN">
@@
 <vertex x="6.985" y="55.245"/>
 <vertex x="6.985" y="50.8"/>
-<vertex x="1.905" y="45.72"/>
-<vertex x="1.905" y="40.005"/>
-<vertex x="4.445" y="37.465"/>
+<vertex x="2.54" y="46.355"/>
+<vertex x="2.54" y="40.005"/>
+<vertex x="4.445" y="38.1"/>
 <vertex x="4.445" y="36.195"/>
 <vertex x="5.715" y="36.195"/>
 <vertex x="5.715" y="38.735"/>
-<vertex x="3.81" y="40.64"/>
-<vertex x="3.81" y="45.72"/>
+<vertex x="4.445" y="40.005"/>
+<vertex x="4.445" y="46.355"/>
 <vertex x="6.35" y="48.26"/>
 <vertex x="8.89" y="48.26"/>
@@
 <contactref element="J2" pad="B7"/>
 <contactref element="U4" pad="15"/>
-<wire x1="38.815" y1="24.51" x2="62.865" y2="26.67" width="0" layer="19" extent="1-1"/>
+<wire x1="62.865" y1="26.67" x2="61.595" y2="27.94" width="0.2032" layer="1"/>
+<wire x1="61.595" y1="27.94" x2="58.42" y2="27.94" width="0.2032" layer="1"/>
+<wire x1="58.42" y1="27.94" x2="54.61" y2="31.75" width="0.2032" layer="1"/>
+<wire x1="54.61" y1="31.75" x2="41.275" y2="31.75" width="0.2032" layer="1"/>
+<wire x1="41.275" y1="31.75" x2="40.3225" y2="30.7975" width="0.2032" layer="1"/>
+<wire x1="40.3225" y1="30.7975" x2="39.37" y2="29.845" width="0.2032" layer="1"/>
+<wire x1="38.815" y1="24.51" x2="38.815" y2="29.29" width="0.2032" layer="1"/>
+<wire x1="38.815" y1="29.29" x2="39.37" y2="29.845" width="0.2032" layer="1"/>
 </signal>
 <signal name="MOSI">
@@
 <contactref element="R3" pad="2"/>
 <contactref element="J3" pad="1"/>
-<wire x1="5.715" y1="40.815" x2="6.525" y2="40.815" width="0.2032" layer="1"/>
-<wire x1="6.525" y1="40.815" x2="7.62" y2="41.91" width="0.2032" layer="1"/>
-<wire x1="17.145" y1="41.91" x2="17.78" y2="42.545" width="0.2032" layer="1"/>
+<wire x1="5.715" y1="40.815" x2="5.89" y2="40.815" width="0.2032" layer="1"/>
+<wire x1="5.89" y1="40.815" x2="6.35" y2="41.275" width="0.2032" layer="1"/>
+<wire x1="16.51" y1="41.275" x2="17.78" y2="42.545" width="0.2032" layer="1"/>
 <wire x1="17.78" y1="42.545" x2="17.78" y2="44.185" width="0.2032" layer="1"/>
-<wire x1="13.065" y1="43.0192" x2="13.065" y2="41.91" width="0.2032" layer="1"/>
-<wire x1="17.145" y1="41.91" x2="13.065" y2="41.91" width="0.2032" layer="1"/>
-<wire x1="13.065" y1="41.91" x2="7.62" y2="41.91" width="0.2032" layer="1"/>
+<wire x1="13.065" y1="43.0192" x2="13.065" y2="41.275" width="0.2032" layer="1"/>
+<wire x1="16.51" y1="41.275" x2="13.065" y2="41.275" width="0.2032" layer="1"/>
+<wire x1="13.065" y1="41.275" x2="6.35" y2="41.275" width="0.2032" layer="1"/>
 </signal>
 <signal name="PI_SCK">
@@
 <contactref element="U2" pad="1"/>
 <contactref element="C4" pad="1"/>
-<wire x1="14.065" y1="45.8962" x2="15.7862" y2="45.8962" width="0.2032" layer="1"/>
-<wire x1="15.7862" y1="45.8962" x2="15.875" y2="45.985" width="0.2032" layer="1"/>
-<wire x1="28.31" y1="44.45" x2="28.31" y2="41.9901" width="0.4064" layer="1"/>
-<wire x1="28.31" y1="41.9901" x2="28.26" y2="41.9401" width="0.4064" layer="1"/>
-<wire x1="28.06" y1="46.99" x2="28.69" y2="51.23" width="0" layer="19" extent="1-1"/>
-<wire x1="28.31" y1="44.45" x2="28.06" y2="46.99" width="0" layer="19" extent="1-1"/>
-<wire x1="15.875" y1="45.985" x2="28.06" y2="46.99" width="0" layer="19" extent="1-1"/>
-<wire x1="8.37" y1="51.23" x2="14.065" y2="45.8962" width="0" layer="19" extent="1-1"/>
-<wire x1="53.71" y1="9.525" x2="28.26" y2="41.9401" width="0" layer="19" extent="1-1"/>
+<via x="26.67" y="46.99" extent="1-16" drill="0.6"/>
+<via x="25.4" y="46.99" extent="1-16" drill="0.6"/>
+<polygon width="0.2032" layer="1" isolate="0.2032" rank="2">
+<vertex x="24.765" y="47.625"/>
+<vertex x="24.765" y="46.355"/>
+<vertex x="27.305" y="46.355"/>
+<vertex x="27.94" y="45.72"/>
+<vertex x="27.94" y="41.91"/>
+<vertex x="28.575" y="41.91"/>
+<vertex x="28.575" y="47.625"/>
+</polygon>
+<via x="14.605" y="46.99" extent="1-16" drill="0.6"/>
+<polygon width="0.2032" layer="1" isolate="0.2032" rank="2">
+<vertex x="13.97" y="47.625"/>
+<vertex x="13.97" y="45.72"/>
+<vertex x="16.51" y="45.72"/>
+<vertex x="16.51" y="46.355"/>
+<vertex x="15.24" y="47.625"/>
+</polygon>
+<wire x1="14.605" y1="46.99" x2="26.67" y2="46.99" width="0.4064" layer="16"/>
+<wire x1="14.605" y1="46.99" x2="12.61" y2="46.99" width="0.4064" layer="16"/>
+<wire x1="12.61" y1="46.99" x2="8.37" y2="51.23" width="0.4064" layer="16"/>
+<wire x1="28.69" y1="51.23" x2="28.69" y2="47.62" width="0.4064" layer="1"/>
+<wire x1="28.69" y1="47.62" x2="28.06" y2="46.99" width="0.4064" layer="1"/>
+<wire x1="28.26" y1="41.9401" x2="53.71" y2="9.525" width="0" layer="19" extent="1-1"/>
 </signal>
 <signal name="P_SDA">
@@
 <contactref element="R3" pad="1"/>
 <contactref element="U2" pad="2"/>
-<wire x1="13.565" y1="45.8962" x2="13.565" y2="46.99" width="0.2032" layer="1"/>
-<wire x1="13.565" y1="46.99" x2="13.565" y2="51.115" width="0.2032" layer="1"/>
+<wire x1="13.565" y1="45.8962" x2="13.565" y2="48.26" width="0.2032" layer="1"/>
+<wire x1="13.565" y1="48.26" x2="13.565" y2="51.115" width="0.2032" layer="1"/>
 <wire x1="13.565" y1="51.115" x2="13.45" y2="51.23" width="0.2032" layer="1"/>
 <wire x1="17.78" y1="45.985" x2="17.515" y2="45.985" width="0.2032" layer="1"/>
-<wire x1="17.515" y1="45.985" x2="16.51" y2="46.99" width="0.2032" layer="1"/>
-<wire x1="16.51" y1="46.99" x2="13.565" y2="46.99" width="0.2032" layer="1"/>
+<wire x1="17.515" y1="45.985" x2="15.24" y2="48.26" width="0.2032" layer="1"/>
+<wire x1="15.24" y1="48.26" x2="13.565" y2="48.26" width="0.2032" layer="1"/>
 </signal>
 <signal name="!RST!">

Commit message: Finalize routing on the Raspberry PI-compatible Application Module. 5V net is not routed, but is not used on the module so not required.
Parts:
- moved R6 44.3 mm to (33.0, 48.3)
- moved S1 2.01 mm to (51.4, 3.17)
Connections:
- net BTN: now also J1.29
Routing:
- net BTN: track 0.00 -> 78.6 mm, vias 0 -> 2
- net !RST!: track 0.00 -> 48.6 mm
- net LINT: track 0.00 -> 44.5 mm, vias 0 -> 1
- net 3.3V: track 30.2 -> 49.2 mm, vias 2 -> 4
- net 3V_PI: track 24.6 -> 28.0 mm
- net VBAT: track 0.00 -> 2.54 mm
- added copper zone on layer 1, net 3.3V
Changed lines of the file:
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@@
 <attribute name="NAME" x="7.747" y="47.371" size="0.6096" layer="25" font="vector" ratio="15" rot="R180"/>
 </element>
-<element name="R6" library="SparkFun-Passives" package="0805" value="10K" x="54.61" y="9.525" smashed="yes" rot="R180">
-<attribute name="NAME" x="55.372" y="8.6995" size="0.6096" layer="25" ratio="15" rot="R180"/>
-<attribute name="VALUE" x="55.626" y="10.922" size="0.6096" layer="27" ratio="15" rot="R180"/>
-</element>
-<element name="S1" library="HAB" package="TACTILE-PTH-THIN" value="POWER" x="53.34" y="2.54" smashed="yes">
-<attribute name="NAME" x="55.88" y="3.81" size="0.6096" layer="25" ratio="15"/>
+<element name="R6" library="SparkFun-Passives" package="0805" value="10K" x="33.02" y="48.26" smashed="yes" rot="R180">
+<attribute name="NAME" x="33.782" y="47.4345" size="0.6096" layer="25" ratio="15" rot="R180"/>
+<attribute name="VALUE" x="34.036" y="49.657" size="0.6096" layer="27" ratio="15" rot="R180"/>
+</element>
+<element name="S1" library="HAB" package="TACTILE-PTH-THIN" value="POWER" x="51.435" y="3.175" smashed="yes">
+<attribute name="NAME" x="53.975" y="4.445" size="0.6096" layer="25" ratio="15"/>
 </element>
 <element name="U$1" library="HAB" package="MSFT_LOGO" value="" x="37.465" y="34.29" rot="MR0"/>
@@
 <wire x1="25.03" y1="40.005" x2="26.035" y2="40.005" width="0.4064" layer="1"/>
 <via x="26.035" y="40.005" extent="1-16" drill="0.5"/>
-<wire x1="26.035" y1="40.005" x2="17.78" y2="40.005" width="0.4064" layer="16"/>
-<wire x1="17.78" y1="40.005" x2="15.24" y2="42.545" width="0.4064" layer="16"/>
+<wire x1="26.035" y1="40.005" x2="17.78" y2="40.005" width="0.6096" layer="16"/>
+<wire x1="17.78" y1="40.005" x2="15.24" y2="42.545" width="0.6096" layer="16"/>
 <wire x1="14.065" y1="43.0192" x2="14.7658" y2="43.0192" width="0.3048" layer="1"/>
 <wire x1="14.7658" y1="43.0192" x2="15.24" y2="42.545" width="0.3048" layer="1"/>
 <via x="15.24" y="42.545" extent="1-16" drill="0.5"/>
-<wire x1="40.815" y1="8.51" x2="62.865" y2="36.83" width="0" layer="19" extent="1-1"/>
-<wire x1="26.035" y1="40.005" x2="40.815" y2="8.51" width="0" layer="19" extent="1-1"/>
+<polygon width="0.2032" layer="1" isolate="0.3048" rank="2">
+<vertex x="42.545" y="40.64"/>
+<vertex x="42.545" y="39.37"/>
+<vertex x="61.595" y="39.37"/>
+<vertex x="62.23" y="38.735"/>
+<vertex x="62.23" y="36.195"/>
+<vertex x="62.865" y="36.195"/>
+<vertex x="63.5" y="35.56"/>
+<vertex x="63.5" y="9.525"/>
+<vertex x="62.23" y="8.255"/>
+<vertex x="58.42" y="8.255"/>
+<vertex x="56.515" y="6.35"/>
+<vertex x="56.515" y="2.54"/>
+<vertex x="55.88" y="1.905"/>
+<vertex x="43.18" y="1.905"/>
+<vertex x="41.91" y="3.175"/>
+<vertex x="41.91" y="5.08"/>
+<vertex x="41.275" y="5.08"/>
+<vertex x="41.275" y="1.905"/>
+<vertex x="42.545" y="0.635"/>
+<vertex x="57.785" y="0.635"/>
+<vertex x="57.785" y="5.715"/>
+<vertex x="59.055" y="6.985"/>
+<vertex x="64.77" y="6.985"/>
+<vertex x="64.77" y="40.64"/>
+</polygon>
+<via x="43.18" y="40.005" extent="1-16" drill="0.7"/>
+<via x="45.085" y="40.005" extent="1-16" drill="0.7"/>
+<wire x1="26.035" y1="40.005" x2="45.085" y2="40.005" width="0.6096" layer="16"/>
 </signal>
 <signal name="5V">
@@
 <contactref element="S1" pad="2"/>
 <contactref element="R6" pad="1"/>
-<wire x1="56.5912" y1="2.54" x2="55.51" y2="9.525" width="0" layer="19" extent="1-1"/>
+<contactref element="J1" pad="29"/>
+<wire x1="33.92" y1="48.26" x2="40.005" y2="48.26" width="0.2032" layer="1"/>
+<wire x1="40.005" y1="48.26" x2="43.18" y2="48.26" width="0.2032" layer="1"/>
+<wire x1="43.18" y1="48.26" x2="43.93" y2="49.01" width="0.2032" layer="1"/>
+<wire x1="43.93" y1="51.23" x2="43.93" y2="49.01" width="0.2032" layer="1"/>
+<via x="55.88" y="10.795" extent="1-16" drill="0.5"/>
+<wire x1="55.88" y1="10.795" x2="53.975" y2="12.7" width="0.2032" layer="16"/>
+<wire x1="53.975" y1="12.7" x2="37.465" y2="12.7" width="0.2032" layer="16"/>
+<wire x1="37.465" y1="12.7" x2="34.925" y2="15.24" width="0.2032" layer="16"/>
+<wire x1="34.925" y1="15.24" x2="34.925" y2="29.845" width="0.2032" layer="16"/>
+<wire x1="34.925" y1="29.845" x2="40.005" y2="34.925" width="0.2032" layer="16"/>
+<via x="40.005" y="34.925" extent="1-16" drill="0.5"/>
+<wire x1="40.005" y1="34.925" x2="40.005" y2="48.26" width="0.2032" layer="1"/>
+<wire x1="55.88" y1="10.795" x2="55.88" y2="4.3688" width="0.2032" layer="1"/>
+<wire x1="55.88" y1="4.3688" x2="54.6862" y2="3.175" width="0.2032" layer="1"/>
 </signal>
 <signal name="TX">
@@
 <wire x1="23.495" y1="48.895" x2="22.352" y2="50.038" width="0.2032" layer="16"/>
 <wire x1="22.352" y1="50.038" x2="22.352" y2="51.943" width="0.2032" layer="16"/>
-<wire x1="22.352" y1="51.943" x2="21.717" y2="52.578" width="0.2032" layer="16"/>
-<wire x1="21.717" y1="52.578" x2="19.722" y2="52.578" width="0.2032" layer="16"/>
-<wire x1="19.722" y1="52.578" x2="18.53" y2="53.77" width="0.2032" layer="16"/>
+<wire x1="22.352" y1="51.943" x2="21.844" y2="52.451" width="0.2032" layer="16"/>
+<wire x1="21.844" y1="52.451" x2="19.849" y2="52.451" width="0.2032" layer="16"/>
+<wire x1="19.849" y1="52.451" x2="18.53" y2="53.77" width="0.2032" layer="16"/>
 </signal>
 <signal name="UART_EN">
@@
 <contactref element="J2" pad="A1"/>
 <contactref element="J2" pad="A2"/>
-<wire x1="2.54" y1="19.05" x2="5.08" y2="19.05" width="0" layer="19" extent="1-1"/>
+<wire x1="2.54" y1="19.05" x2="5.08" y2="19.05" width="1.27" layer="1"/>
 </signal>
 <signal name="VS">
@@
 <wire x1="14.605" y1="46.99" x2="12.61" y2="46.99" width="0.4064" layer="16"/>
 <wire x1="12.61" y1="46.99" x2="8.37" y2="51.23" width="0.4064" layer="16"/>
-<wire x1="28.69" y1="51.23" x2="28.69" y2="47.62" width="0.4064" layer="1"/>
+<wire x1="28.69" y1="51.23" x2="28.69" y2="48.26" width="0.4064" layer="1"/>
+<wire x1="28.69" y1="48.26" x2="28.69" y2="47.62" width="0.4064" layer="1"/>
 <wire x1="28.69" y1="47.62" x2="28.06" y2="46.99" width="0.4064" layer="1"/>
-<wire x1="28.26" y1="41.9401" x2="53.71" y2="9.525" width="0" layer="19" extent="1-1"/>
+<wire x1="32.12" y1="48.26" x2="28.69" y2="48.26" width="0.4064" layer="1"/>
 </signal>
 <signal name="P_SDA">
@@
 <contactref element="U4" pad="4"/>
 <contactref element="J2" pad="B10"/>
-<wire x1="42.815" y1="8.51" x2="60.325" y2="29.21" width="0" layer="19" extent="1-1"/>
+<wire x1="60.325" y1="29.21" x2="59.055" y2="29.21" width="0.2032" layer="1"/>
+<wire x1="59.055" y1="29.21" x2="55.245" y2="33.02" width="0.2032" layer="1"/>
+<wire x1="55.245" y1="33.02" x2="41.275" y2="33.02" width="0.2032" layer="1"/>
+<wire x1="41.275" y1="33.02" x2="37.846" y2="29.591" width="0.2032" layer="1"/>
+<wire x1="42.815" y1="8.51" x2="42.815" y2="13.7" width="0.2032" layer="1"/>
+<wire x1="42.815" y1="13.7" x2="37.846" y2="18.669" width="0.2032" layer="1"/>
+<wire x1="37.846" y1="18.669" x2="37.846" y2="29.591" width="0.2032" layer="1"/>
 </signal>
 <signal name="LINT">
 <contactref element="U4" pad="5"/>
 <contactref element="J2" pad="B9"/>
-<wire x1="44.815" y1="8.51" x2="62.865" y2="29.21" width="0" layer="19" extent="1-1"/>
+<wire x1="62.865" y1="29.21" x2="64.135" y2="27.94" width="0.2032" layer="16"/>
+<wire x1="64.135" y1="27.94" x2="64.135" y2="8.255" width="0.2032" layer="16"/>
+<wire x1="64.135" y1="8.255" x2="62.865" y2="6.985" width="0.2032" layer="16"/>
+<wire x1="62.865" y1="6.985" x2="54.61" y2="6.985" width="0.2032" layer="16"/>
+<wire x1="54.61" y1="6.985" x2="53.34" y2="5.715" width="0.2032" layer="16"/>
+<via x="53.34" y="5.715" extent="1-16" drill="0.5"/>
+<wire x1="53.34" y1="5.715" x2="45.085" y2="5.715" width="0.2032" layer="1"/>
+<wire x1="44.815" y1="8.51" x2="44.815" y2="5.985" width="0.2032" layer="1"/>
+<wire x1="44.815" y1="5.985" x2="45.085" y2="5.715" width="0.2032" layer="1"/>
 </signal>
 <signal name="ANT">
