File: hardware/tmod-base.sch (EAGLE design)
At the start: 97 parts, among them IC1 TPS70933, IC2 RA02, IC3 STM32L052C8T6, IC4 HX1, IC5 LMP7702, IC6 TPS62160, IC7 TPS70933, IC8 TPS22918, J1 DNP, J2 GPS1, J3 TEMP, J4 POWER, J5 GPS2, J6 MICRO-SD_CARD_SOCKET, J7 RASPBERRYPI-GPIO, U1 BME280, U2 ADXL345, Y1 8M, Y2 32768

Commit message: Initial route for HAB v3 modular base board
Parts:
- removed R2, R26, R27: 10K, SparkFun-Passives:RESISTOR0805-RES
- removed R23: 82K, SparkFun-Passives:RESISTOR0805-RES
- added C31: 1n, SparkFun-Passives:CAP0805
- added D12: 5.6V, SparkFun-DiscreteSemi:DIODE-ZENER5.6V
- added J8: STACK2, SparkFun-Connectors:CONN_08X2
- C23: value 100u -> 150u
- C26: value 1u -> 3.3n
- C28: value 10u -> 1u
- C29: value 0.1u -> 10u
- C30: value 1n -> 0.1u
- IC2: value RA02 -> INA219SOT; device HAB:RA02 -> HAB:INA219SOT
- IC6: value TPS62160 -> TPS62143; device HAB:TPS62160 -> HAB:TPS62140
- J7: value RASPBERRYPI-GPIO -> STACK1; device HAB:RASPBERRYPI-GPIO -> SparkFun-Connectors:CONN_08X2
- L1: device HAB:INDUCTOR1206 -> HAB:INDUCTOR0805
- L2: device HAB:INDUCTOR1008 -> HAB:INDUCTORMPIA4012V2
- R21: value 10K -> 100K
- R22: value 430K -> 0.01; device SparkFun-Passives:RESISTOR0805-RES -> SparkFun-Resistors:0.1OHM-1210-1/2W-1%
- R24: value 430K -> 10K
- R25: value 100K -> 10K
- renumbered IC7 to IC10, U1 to IC9
Connections:
- removed net !LORA_IRQ!: IC2.DIO0
- removed net !LORA_RST!: IC2.!RESET!, R2.1
- removed net 3V_PI: J7.3.3V@1
- removed net 3V_PI2: J7.3.3V@17
- removed net FB5: IC6.FB, R22.1, R23.2
- removed net MISO: D6.C, IC2.MISO, IC3.PB4, J6.DO
- removed net MOSI: D11.C, IC2.MOSI, IC3.PB5, J6.DI
- removed net R_CS0: J7.CE0
- removed net R_CS1: J7.CE1
- removed net R_MISO: J7.MISO
- removed net R_MOSI: J7.MOSI
- removed net R_SCK: J7.SCLK
- removed net SCK: D10.C, IC2.SCK, IC3.PB3, J6.SCK
- removed net U_RX: IC3.PB6
- removed net VDIV: IC3.PA5, R24.1, R25.2
- new net MISO1: IC3.PB4, J6.DO
- new net MISO2: D6.C, IC3.PB14, J8.6
- new net MOSI1: IC3.PB5, J6.DI
- new net MOSI2: D11.C, IC3.PB15, J8.5
- new net RFU1: IC3.PA5
- new net RFU2: IC3.PB2
- new net SCK1: IC3.PB3, J6.SCK
- new net SCK2: D10.C, IC3.PB13, J8.2
- new net SS5: C26.1, IC6.SS
- new net VIN: IC2.IN+, J4.1, R22.2
- net 3.3V: now also J8.15, J8.3, R25.2; no longer R2.2, R27.2
- net 5V: now also C30.1, D4.C, J7.13; no longer C28.1, D5.C, R22.2
- net 5V_PI: now also J7.15; no longer J7.5V@2, J7.5V@4
- net CT: now also C31.1; no longer C30.1
- net GND: now also C31.2, D12.A, IC2.A0, IC2.A1, IC6.AGND, IC6.DEF, IC6.FB, IC6.FSW, IC6.PGND, J7.14, J7.16, J7.4, J7.9, J8.1, J8.12, J8.13, J8.4, J8.8, R24.2; no longer IC1.NC/FB, IC6.GND, J7.GND@14, J7.GND@20, J7.GND@25, J7.GND@6, J7.GND@9, R23.1, R25.1, R26.2
- net GPSRX1: now also IC3.PA10; no longer IC3.PB11
- net GPSRX2: now also IC3.PB11; no longer IC3.PA10
- net GPSTX1: now also IC3.PA9; no longer IC3.PB10
- net GPSTX2: now also IC3.PB10; no longer IC3.PA9
- net K_PI: now also R24.1; no longer R26.1
- net LCS: now also D12.C, IC3.PB12, J8.7; no longer IC2.!SS!, IC3.PB7
- net R_RX: now also J7.11, R25.1; no longer J7.RXI, R27.1
- net R_TX: now also J7.12; no longer J7.TXO
- net SCL: now also IC2.SCL, J8.14
- net SDA: now also IC2.SDA, J8.16
- net SW5: now also IC6.SW; no longer IC6.OUT
- net TEMP: now also IC3.PB6; no longer IC3.PA8
- net VBAT: now also IC2.IN-, IC6.AVIN, IC6.PVIN, J7.1, J7.2, R22.1; no longer IC6.VIN, J4.1, R24.2
- net VS: now also C28.1, D5.C, J8.11; no longer C26.1, D4.C
Other:
- note added: "L1: 732-1620-1-ND L2: 283-4729-1-ND C27, C29: 1276-2890-1-ND C23: P15450CT-ND D1, D4-D11: DESD5V0U1BA-7DICT-ND"
- note added: "SAM1196-08-ND"
- note removed: "L1: CVH252009-2R2MCT-ND C19, C20: 1276-2890-1-ND C21: 493-10772-1-ND D3: CDSOD323-T15SCT-ND D1, D4-D11: DESD5V0U1BA-7DICT-ND"
- moved on the sheet: C10, C11, C26, C27, C28, C29, C30, D4, D5, R22, R24, R25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

Commit message: Add silkscreen to HAB base board
Parts:
- D2: value GREEN -> POWER
- LED1: value COM-10866 -> STATUS
Connections:
- net 3.3V: no longer J8.3
- net 5V: now also J8.3
Changed lines of the file:
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@@
 <part name="GND32" library="SparkFun-Aesthetics" deviceset="GND" device=""/>
 <part name="R20" library="SparkFun-Passives" deviceset="RESISTOR" device="0805-RES" value="10K"/>
-<part name="LED1" library="SparkFun-LED" deviceset="LED-TRICOLOR-5050" device="NO_IC" value="COM-10866"/>
+<part name="LED1" library="SparkFun-LED" deviceset="LED-TRICOLOR-5050" device="NO_IC" value="STATUS"/>
 <part name="SUPPLY15" library="SparkFun-Aesthetics" deviceset="5V" device=""/>
 <part name="R8" library="SparkFun-Passives" deviceset="RESISTOR" device="0805-RES" value="470"/>
@@
 <part name="SUPPLY13" library="SparkFun-Aesthetics" deviceset="5V" device=""/>
 <part name="GND20" library="SparkFun-Aesthetics" deviceset="GND" device=""/>
-<part name="D2" library="SparkFun-LED" deviceset="LED-GREEN" device="0603" value="GREEN"/>
+<part name="D2" library="SparkFun-LED" deviceset="LED-GREEN" device="0603" value="POWER"/>
 <part name="IC6" library="HAB" deviceset="TPS62140" device="" value="TPS62143"/>
 <part name="C26" library="SparkFun-Passives" deviceset="CAP" device="0805" value="3.3n"/>
@@
 <label x="419.1" y="86.36" size="1.778" layer="95"/>
 </segment>
-<segment>
-<pinref part="J8" gate="G$1" pin="3"/>
-<wire x1="419.1" y1="101.6" x2="429.26" y2="101.6" width="0.1524" layer="91"/>
-<label x="419.1" y="101.6" size="1.778" layer="95"/>
-</segment>
 </net>
 <net name="VDDA" class="0">
@@
 <label x="419.1" y="119.38" size="1.778" layer="95"/>
 </segment>
+<segment>
+<pinref part="J8" gate="G$1" pin="3"/>
+<wire x1="419.1" y1="101.6" x2="429.26" y2="101.6" width="0.1524" layer="91"/>
+<label x="419.1" y="101.6" size="1.778" layer="95"/>
+</segment>
 </net>

Commit message: Started work on Pi and Edison example application cards, neither is complete
Parts:
- removed J8: STACK2, SparkFun-Connectors:CONN_08X2
- J7: value STACK1 -> HAB-EXP; device SparkFun-Connectors:CONN_08X2 -> HAB:HAB-EXP
Connections:
- new net RSV7: IC3.PB6, J7R.RSV7
- net !RST!: now also J7R.!RST!
- net 3.3V: now also J7R.3.3V; no longer J8.15
- net 5V: now also J7L.5V, J7R.5V; no longer J7.13, J8.3
- net 5V_PI: now also J7L.5V_SW; no longer J7.15
- net GND: now also J7L.GND, J7R.GND; no longer J7.14, J7.16, J7.4, J7.9, J8.1, J8.12, J8.13, J8.4, J8.8
- net LCS: now also J7R.CS; no longer J8.7
- net MISO2: now also J7R.MISO; no longer J8.6
- net MOSI2: now also J7R.MOSI; no longer J8.5
- net R_RX: now also J7L.RXI; no longer J7.11
- net R_TX: now also J7L.TXO; no longer J7.12
- net SCK2: now also J7R.SCK; no longer J8.2
- net SCL: now also J7R.SCL; no longer J8.14
- net SDA: now also J7R.SDA; no longer J8.16
- net TEMP: now also IC3.PB7; no longer IC3.PB6
- net VBAT: now also J7L.VBAT; no longer J7.1, J7.2
- net VS: now also J7R.VS; no longer J8.11
Other:
- note removed: "SAM1196-08-ND"
- moved on the sheet: R25

Commit message: Route out RSV5 and RSV6 to microcontroller pins
Parts:
- added D13, D14: 5.6V, SparkFun-DiscreteSemi:DIODE-ZENER5.6V
Connections:
- removed net RFU1: IC3.PA5
- removed net RFU2: IC3.PB2
- new net RSV5: D13.C, IC3.PB2, J7L.RSV5
- new net RSV6: D14.C, IC3.PA5, J7L.RSV6
- net GND: now also D13.A, D14.A
Other:
- moved on the sheet: R25
Changed lines of the file:
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@@
 <part name="GND49" library="SparkFun-Aesthetics" deviceset="GND" device=""/>
 <part name="J7" library="HAB" deviceset="HAB-EXP" device=""/>
+<part name="D13" library="SparkFun-DiscreteSemi" deviceset="DIODE-ZENER" device="5.6V" value="5.6V"/>
+<part name="D14" library="SparkFun-DiscreteSemi" deviceset="DIODE-ZENER" device="5.6V" value="5.6V"/>
+<part name="GND46" library="SparkFun-Aesthetics" deviceset="GND" device=""/>
 </parts>
 <sheets>
@@
 <instance part="R17" gate="G$1" x="228.6" y="170.18" rot="R90"/>
 <instance part="R19" gate="G$1" x="238.76" y="170.18" rot="R90"/>
-<instance part="R25" gate="G$1" x="462.28" y="121.92" rot="R90"/>
-<instance part="SUPPLY24" gate="G$1" x="462.28" y="129.54"/>
+<instance part="R25" gate="G$1" x="500.38" y="121.92" rot="R90"/>
+<instance part="SUPPLY24" gate="G$1" x="500.38" y="129.54"/>
 <instance part="GND39" gate="1" x="431.8" y="152.4"/>
 <instance part="SUPPLY23" gate="G$1" x="431.8" y="175.26"/>
@@
 <instance part="J7" gate="L" x="436.88" y="121.92"/>
 <instance part="J7" gate="R" x="436.88" y="88.9"/>
+<instance part="D13" gate="G$1" x="459.74" y="121.92" smashed="yes" rot="R90">
+<attribute name="NAME" x="462.28" y="122.4026" size="1.778" layer="95"/>
+<attribute name="VALUE" x="462.28" y="119.6086" size="1.778" layer="96"/>
+</instance>
+<instance part="D14" gate="G$1" x="469.9" y="121.92" smashed="yes" rot="R90">
+<attribute name="NAME" x="472.44" y="122.4026" size="1.778" layer="95"/>
+<attribute name="VALUE" x="472.44" y="119.6086" size="1.778" layer="96"/>
+</instance>
+<instance part="GND46" gate="1" x="459.74" y="111.76"/>
 </instances>
 <busses>
@@
 <pinref part="J7" gate="R" pin="GND"/>
 </segment>
+<segment>
+<pinref part="GND46" gate="1" pin="GND"/>
+<pinref part="D13" gate="G$1" pin="A"/>
+<wire x1="459.74" y1="114.3" x2="459.74" y2="116.84" width="0.1524" layer="91"/>
+<pinref part="D14" gate="G$1" pin="A"/>
+<wire x1="459.74" y1="116.84" x2="459.74" y2="119.38" width="0.1524" layer="91"/>
+<wire x1="459.74" y1="116.84" x2="469.9" y2="116.84" width="0.1524" layer="91"/>
+<wire x1="469.9" y1="116.84" x2="469.9" y2="119.38" width="0.1524" layer="91"/>
+<junction x="459.74" y="116.84"/>
+</segment>
 </net>
 <net name="3.3V" class="0">
@@
 <segment>
 <pinref part="R25" gate="G$1" pin="2"/>
-<wire x1="462.28" y1="127" x2="462.28" y2="129.54" width="0.1524" layer="91"/>
+<wire x1="500.38" y1="127" x2="500.38" y2="129.54" width="0.1524" layer="91"/>
 <pinref part="SUPPLY24" gate="G$1" pin="3.3V"/>
 </segment>
@@
 <net name="R_RX" class="0">
 <segment>
-<label x="452.12" y="114.3" size="1.778" layer="95"/>
+<label x="490.22" y="114.3" size="1.778" layer="95"/>
 <pinref part="R25" gate="G$1" pin="1"/>
-<wire x1="452.12" y1="114.3" x2="462.28" y2="114.3" width="0.1524" layer="91"/>
-<wire x1="462.28" y1="114.3" x2="462.28" y2="116.84" width="0.1524" layer="91"/>
+<wire x1="490.22" y1="114.3" x2="500.38" y2="114.3" width="0.1524" layer="91"/>
+<wire x1="500.38" y1="114.3" x2="500.38" y2="116.84" width="0.1524" layer="91"/>
 </segment>
 <segment>
@@
 </segment>
 </net>
-<net name="RFU2" class="0">
+<net name="RSV7" class="0">
+<segment>
+<pinref part="J7" gate="R" pin="RSV7"/>
+<wire x1="454.66" y1="93.98" x2="449.58" y2="93.98" width="0.1524" layer="91"/>
+<label x="452.12" y="93.98" size="1.778" layer="95"/>
+</segment>
+<segment>
+<pinref part="IC3" gate="G$1" pin="PB6"/>
+<wire x1="68.58" y1="86.36" x2="68.58" y2="91.44" width="0.1524" layer="91"/>
+<label x="68.58" y="88.9" size="1.778" layer="95" rot="R90"/>
+</segment>
+</net>
+<net name="RSV6" class="0">
+<segment>
+<pinref part="J7" gate="L" pin="RSV6"/>
+<label x="452.12" y="129.54" size="1.778" layer="95"/>
+<wire x1="449.58" y1="129.54" x2="469.9" y2="129.54" width="0.1524" layer="91"/>
+<pinref part="D14" gate="G$1" pin="C"/>
+<wire x1="469.9" y1="129.54" x2="469.9" y2="124.46" width="0.1524" layer="91"/>
+</segment>
+<segment>
+<pinref part="IC3" gate="G$1" pin="PA5"/>
+<wire x1="60.96" y1="30.48" x2="60.96" y2="40.64" width="0.1524" layer="91"/>
+<label x="60.96" y="30.48" size="1.778" layer="95" rot="R90"/>
+</segment>
+</net>
+<net name="RSV5" class="0">
+<segment>
+<pinref part="J7" gate="L" pin="RSV5"/>
+<label x="452.12" y="127" size="1.778" layer="95"/>
+<pinref part="D13" gate="G$1" pin="C"/>
+<wire x1="459.74" y1="124.46" x2="459.74" y2="127" width="0.1524" layer="91"/>
+<wire x1="459.74" y1="127" x2="449.58" y2="127" width="0.1524" layer="91"/>
+</segment>
 <segment>
 <pinref part="IC3" gate="G$1" pin="PB2"/>
@@
 </segment>
 </net>
-<net name="RFU1" class="0">
-<segment>
-<pinref part="IC3" gate="G$1" pin="PA5"/>
-<wire x1="60.96" y1="30.48" x2="60.96" y2="40.64" width="0.1524" layer="91"/>
-<label x="60.96" y="30.48" size="1.778" layer="95" rot="R90"/>
-</segment>
-</net>
-<net name="RSV7" class="0">
-<segment>
-<pinref part="J7" gate="R" pin="RSV7"/>
-<wire x1="454.66" y1="93.98" x2="449.58" y2="93.98" width="0.1524" layer="91"/>
-<label x="452.12" y="93.98" size="1.778" layer="95"/>
-</segment>
-<segment>
-<pinref part="IC3" gate="G$1" pin="PB6"/>
-<wire x1="68.58" y1="86.36" x2="68.58" y2="91.44" width="0.1524" layer="91"/>
-<label x="68.58" y="88.9" size="1.778" layer="95" rot="R90"/>
-</segment>
-</net>
