File: hardware/fadic.sch (EAGLE design)
At the start: 97 parts, among them IC1 TPS70933, IC10 TPS70933, IC2 INA219SOT, IC3 STM32L443CCT6, IC4 HX1, IC5 LMP7702, IC6 TPS62143, IC8 TPS22918, IC9 BME280, J1 DNP, J2 GPS1, J3 TEMP, J4 POWER, J5 GPS2, J6 MICRO-SD_CARD_SOCKET, J7 HAB-EXP, U2 ADXL345, Y1 8M, Y2 32768

Commit message: Start work on new automated base station. Add BOM for Pi application board. Fix mirrored INA219 footprint and LED on base board
Parts:
- removed C22, C25, C30: 0.1u, SparkFun-Passives:CAP0805
- removed C23: 150u, SparkFun-Passives:CAP_POLE
- removed C24, C28: 1u, SparkFun-Passives:CAP0805
- removed C26: 3.3n, SparkFun-Passives:CAP0805
- removed C27, C29: 10u, SparkFun-Passives:CAP0805
- removed C31: 1n, SparkFun-Passives:CAP0805
- removed D10, D11, D12, D13, D14, D4, D5, D6, D7, D8, D9: 5.6V, SparkFun-DiscreteSemi:DIODE-ZENER5.6V
- removed FRAME2: FRAME-LETTERNO_PACKAGE, SparkFun-Aesthetics:FRAME-LETTERNO_PACKAGE
- removed IC10: TPS70933, texas:TPS77033
- removed IC6: TPS62143, HAB:TPS62140
- removed IC8: TPS22918, HAB:TPS22918
- removed IC9: BME280, BME280ComponentLibrary:BME280
- removed J4: POWER, HAB:1X02
- removed J7: HAB-EXP, HAB:HAB-EXP
- removed L2: 2.2u, HAB:INDUCTORMPIA4012V2
- removed U2: ADXL345, SparkFun-Sensors:ADXL345
- added R2: 0, SparkFun-Passives:RESISTOR0805-RES
- added R23: DNP, SparkFun-Passives:RESISTOR0805-RES
- added R26: 22K, SparkFun-Passives:RESISTOR0805-RES
- added R27: 22, SparkFun-Passives:RESISTOR0805-RES
- C10: value 0.1u -> 330p
- C11: value 10u -> 0.1u
- C15: value 0.1u -> 10u
- C20: value 1.0u -> 1u
- D3: value 15V -> 5.6V
- IC2: value INA219SOT -> BIM1H; device HAB:INA219SOT -> HAB:BIM1H
- IC4: value HX1 -> LMP7702; device HAB:HX1 -> HAB:LMP7702VSSOP
- J3: value TEMP -> ZX62-B-5PA; device SparkFun-Connectors:CONN_03JST-PTH -> OPL_Connector:MICRO-USB-SMD(ZX62-B-5PA)
- R16: value 4.7K -> 0
- R20: value 10K -> 4.7K
- R21: value 100K -> 22
- R22: value 0.01 -> DNP; device SparkFun-Resistors:0.1OHM-1210-1/2W-1% -> SparkFun-Passives:RESISTOR0805-RES
- R24: value 10K -> 0
- R7: value 10K -> DNP
Connections:
- removed net 5V_PI: IC8.VOUT, J7L.5V_SW
- removed net ADXL_SDO: R20.2, U2.SDO
- removed net BME_SDO: IC9.SDO/ADR, R7.2
- removed net CT: C31.1, IC8.CT
- removed net HXEN: IC3.PA6, IC4.EN, R6.1
- removed net INT: U2.INT1
- removed net INT2: U2.INT2
- removed net K_PI: IC3.PA0, IC8.ON, R24.1
- removed net LCS: D12.C, IC3.PB12, J7R.CS, R4.1
- removed net PG5: IC6.PG, R21.1
- removed net RF_HX1: IC4.RFOUT, J$1.SIGNAL
- removed net RSV5: D13.C, IC3.PB2, J7L.RSV5
- removed net RSV6: D14.C, IC3.PA5, J7L.RSV6
- removed net RSV7: IC3.PB6, J7R.RSV7
- removed net R_RX: IC3.PA3, J7L.RXI, R25.1
- removed net R_TX: IC3.PA2, J7L.TXO
- removed net SS5: C26.1, IC6.SS
- removed net SW5: IC6.SW, L2.1
- removed net TEMP: D8.C, IC3.PB7, J3.2, R16.1
- removed net VBAT: C23.+, C24.1, D3.C, IC2.IN-, IC6.AVIN, IC6.EN, IC6.PVIN, J7L.VBAT, R22.1
- removed net VIN: IC2.IN+, J4.1, R22.2
- removed net VS: C15.1, C20.1, C22.1, C28.1, D5.C, IC10.OUT, IC9.!CS, IC9.VDD, IC9.VDDIO, J3.3, J7R.VS, R16.2, R17.2, R19.2, U2.CS, U2.VDD, U2.VS
- new net ADC: IC3.PA0, IC4B.OUT, R24.2
- new net AF: IC2.AF, R7.1
- new net BIMRX: IC2.!RXE!, IC3.PA5, R6.1
- new net BIMTX: IC2.!TXE!, IC3.PA6, R20.1
- new net D+: IC3.PA12, R27.2
- new net D-: IC3.PA11, R21.2
- new net GPSRX: IC3.PB11
- new net GPSTX: IC3.PB10
- new net IRQ1: IC3.PB6
- new net IRQ2: IC3.PB7
- new net LCS1: IC3.PB12, R4.1
- new net LCS2: IC3.PA8
- new net LP3: IC4A.OUT, R2.2, R25.2
- new net LP4: IC4B.+IN, R25.1, R26.2
- new net LP5: IC4B.-IN, R24.1
- new net RF_BIM: IC2.ANT, J$1.SIGNAL
- new net RSSI: IC2.RSSI, IC3.PA1
- new net RX: C10.1, R16.2, R7.2
- new net RX1: IC3.PA10
- new net RX2: IC3.PA3
- new net RXD: IC2.RXD, R16.1
- new net TX1: IC3.PA9
- new net TX2: IC3.PA2
- new net USBDM: J3.D-, R21.1
- new net USBDP: J3.D+, R27.1
- new net Z+: C10.2, IC4A.+IN, R22.2, R23.1
- new net Z-: IC4A.-IN, R2.1
- net !RST!: no longer J7R.!RST!
- net 3.3V: now also R17.2, R19.2; no longer C10.1, C11.1, IC2.VCC, J7R.3.3V, R25.2
- net 5V: now also C11.1, C15.1, C20.1, D3.C, IC2.VCC, IC4A.V+, J3.VBUS, R20.2, R23.2; no longer C25.1, C27.1, C29.1, C30.1, D4.C, IC10.IN, IC4.VCC, IC6.VOS, IC8.VIN, J7L.5V, J7R.5V, L2.2, R21.2
- net GND: now also IC4A.V-, J3.GND, J3.SHIELD, R22.1, R26.1; no longer C10.2, C22.2, C23.-, C24.2, C25.2, C26.2, C27.2, C28.2, C29.2, C30.2, C31.2, D10.A, D11.A, D12.A, D13.A, D14.A, D4.A, D5.A, D6.A, D7.A, D8.A, D9.A, IC10.GND, IC2.A0, IC2.A1, IC4.GND, IC6.AGND, IC6.DEF, IC6.FB, IC6.FSW, IC6.PGND, IC8.GND, IC9.GND1, IC9.GND2, J3.1, J4.2, J7L.GND, J7R.GND, R20.1, R24.2, R7.1, U2.GND@2, U2.GND@4, U2.GND@5
- net GPSRX1: no longer IC3.PA10
- net GPSRX2: no longer IC3.PB11
- net GPSTX1: no longer IC3.PA9
- net GPSTX2: no longer IC3.PB10
- net MISO2: no longer D6.C, J7R.MISO
- net MOSI2: no longer D11.C, J7R.MOSI
- net RGND: now also IC2.RFGND; no longer IC4.RFGND
- net SCK2: no longer D10.C, J7R.SCK
- net SCL: no longer D9.C, IC2.SCL, IC9.SCK/SCL, J7R.SCL, U2.SCL
- net SDA: no longer D7.C, IC2.SDA, IC9.SDI/SDA, J7R.SDA, U2.SDA
- net TXD: now also IC2.TXD; no longer IC4.TXD
Other:
- note added: "497-16579-ND"
- note removed: "828-1063-1-ND"
- note removed: "A121350-ND"
- note removed: "Alternative: STM32L433CCT6 497-16579-ND"
- note removed: "L1: 732-1620-1-ND L2: 283-4729-1-ND C27, C29: 1276-2890-1-ND C23: P15450CT-ND D1, D4-D11: DESD5V0U1BA-7DICT-ND"
- moved on the sheet: C10, C11, C15, C16, C20, C21, D3, J6, R16, R20, R21, R22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
